File: Hardware/DomesdayDuplicator-base-DE0Nano/cypress-fx3.sch (KiCad schematic (older format))
At the start: 0 parts

Commit message: Additional schematics for the base-board design + FX3 header parts
Parts:
- added J?: GPIFII_J6, Connector_PinHeader_2.54mm:PinHeader_2x20_P2.54mm_Vertical, symbol Cypress-FX3-Headers:GPIFII_J6
- added J?: GPIFII_J7, Connector_PinHeader_2.54mm:PinHeader_2x20_P2.54mm_Vertical, symbol Cypress-FX3-Headers:GPIFII_J7
Connections:
- new net +5V: J?.3 (USB3_VBUS), J?.4 (USB3_VBUS)
- new net GND: J?.13 (GND), J?.15 (GND), J?.17 (GND), J?.25 (GND), J?.29 (GND), J?.33 (GND), J?.37 (GND), J?.39 (GND), J?.40 (GND), J?.6 (GND)
- new net USB_CTL0: J?.31 (CTL0)
- new net USB_CTL1: J?.29 (CTL1)
- new net USB_CTL10: J?.11 (CTL10)
- new net USB_CTL11: J?.9 (CTL11)
- new net USB_CTL12: J?.7 (CTL12)
- new net USB_CTL2: J?.27 (CTL2)
- new net USB_CTL3: J?.25 (CTL3)
- new net USB_CTL4: J?.23 (CTL4)
- new net USB_CTL5: J?.21 (CTL5)
- new net USB_CTL6: J?.19 (CTL6)
- new net USB_CTL7: J?.17 (CTL7)
- new net USB_CTL8: J?.15 (CTL8)
- new net USB_CTL9: J?.13 (CTL9)
- new net USB_DATA0: J?.38 (DQ0)
- new net USB_DATA1: J?.36 (DQ1)
- new net USB_DATA10: J?.18 (DQ10)
- new net USB_DATA11: J?.16 (DQ11)
- new net USB_DATA12: J?.14 (DQ12)
- new net USB_DATA13: J?.12 (DQ13)
- new net USB_DATA14: J?.10 (DQ14)
- new net USB_DATA15: J?.8 (DQ15)
- new net USB_DATA16: J?.38 (DQ16)
- new net USB_DATA17: J?.36 (DQ17)
- new net USB_DATA18: J?.34 (DQ18)
- new net USB_DATA19: J?.32 (DQ19)
- new net USB_DATA2: J?.34 (DQ2)
- new net USB_DATA20: J?.30 (DQ20)
- new net USB_DATA21: J?.28 (DQ21)
- new net USB_DATA22: J?.26 (DQ22)
- new net USB_DATA23: J?.24 (DQ23)
- new net USB_DATA24: J?.22 (DQ24)
- new net USB_DATA25: J?.20 (DQ25)
- new net USB_DATA26: J?.18 (DQ26)
- new net USB_DATA27: J?.16 (DQ27)
- new net USB_DATA28: J?.12 (DQ28)
- new net USB_DATA29: J?.10 (DQ29)
- new net USB_DATA3: J?.32 (DQ3)
- new net USB_DATA30: J?.8 (DQ30)
- new net USB_DATA31: J?.6 (DQ31)
- new net USB_DATA4: J?.30 (DQ4)
- new net USB_DATA5: J?.28 (DQ5)
- new net USB_DATA6: J?.26 (DQ6)
- new net USB_DATA7: J?.24 (DQ7)
- new net USB_DATA8: J?.22 (DQ8)
- new net USB_DATA9: J?.20 (DQ9)
- new net USB_PCLK: J?.35 (PCLK)
- no-connect marks 0 -> 20

Commit message: Fixes to module and base - added component mapping to base and verified mirrored headers
Parts:
- gave numbers to parts that had none: 2
Changed lines of the file:
@@
 $Descr A4 11693 8268
 encoding utf-8
-Sheet 3 5
+Sheet 3 6
 Title "Domesday Duplicator Base - DE0-Nano/FX3"
 Date "2019-09-02"
@@
 $EndDescr
 $Comp
-L Cypress-FX3-Headers:GPIFII_J6 J?
+L Cypress-FX3-Headers:GPIFII_J6 J301
 U 1 1 5D6E5201
 P 6000 2600
-F 0 "J?" H 6000 3865 50  0000 C CNN
+F 0 "J301" H 6000 3865 50  0000 C CNN
 F 1 "GPIFII_J6" H 6000 3774 50  0000 C CNN
 F 2 "Connector_PinHeader_2.54mm:PinHeader_2x20_P2.54mm_Vertical" H 6000 1450 50  0001 C CNN
@@
 $EndComp
 $Comp
-L Cypress-FX3-Headers:GPIFII_J7 J?
+L Cypress-FX3-Headers:GPIFII_J7 J302
 U 1 1 5D6E89AF
 P 6000 5100
-F 0 "J?" H 6000 6315 50  0000 C CNN
+F 0 "J302" H 6000 6315 50  0000 C CNN
 F 1 "GPIFII_J7" H 6000 6224 50  0000 C CNN
 F 2 "Connector_PinHeader_2.54mm:PinHeader_2x20_P2.54mm_Vertical" H 6000 3900 50  0001 C CNN
@@
 	6900 1800 6900 6050
 Wire Wire Line
-	6900 6350 5100 6350
+	6900 6350 5500 6350
 Connection ~ 5100 6350
 Wire Wire Line
@@
 	5100 4750 5100 4850
 $Comp
-L power:GND #PWR?
+L power:GND #PWR0302
 U 1 1 5D6EFDDB
 P 5100 6600
-F 0 "#PWR?" H 5100 6350 50  0001 C CNN
+F 0 "#PWR0302" H 5100 6350 50  0001 C CNN
 F 1 "GND" H 5105 6427 50  0000 C CNN
 F 2 "" H 5100 6600 50  0001 C CNN
@@
 	6900 1700 6900 1150
 Wire Wire Line
-	6900 1150 5100 1150
+	6900 1150 5500 1150
 Wire Wire Line
 	5100 1150 5100 1700
@@
 	5100 1700 5200 1700
 $Comp
-L power:+5V #PWR?
+L power:+5V #PWR0301
 U 1 1 5D6F37AA
 P 5100 1050
-F 0 "#PWR?" H 5100 900 50  0001 C CNN
+F 0 "#PWR0301" H 5100 900 50  0001 C CNN
 F 1 "+5V" H 5115 1223 50  0000 C CNN
 F 2 "" H 5100 1050 50  0001 C CNN
@@
 Text HLabel 8300 1550 2    50   BiDi ~ 0
 USB_DATA[0..31]
-Wire Bus Line
-	4500 1550 4500 3000
-Wire Bus Line
-	7650 1550 7650 6050
 Text Label 4650 1900 0    50   ~ 0
 USB_CTL12
@@
 Text Label 6950 5950 0    50   ~ 0
 USB_DATA16
+$Comp
+L power:PWR_FLAG #FLG0101
+U 1 1 5D724F63
+P 5500 1050
+F 0 "#FLG0101" H 5500 1125 50  0001 C CNN
+F 1 "PWR_FLAG" H 5500 1223 50  0000 C CNN
+F 2 "" H 5500 1050 50  0001 C CNN
+F 3 "~" H 5500 1050 50  0001 C CNN
+	1    5500 1050
+	1    0    0    -1
+$EndComp
+Wire Wire Line
+	5500 1050 5500 1150
+Connection ~ 5500 1150
+Wire Wire Line
+	5500 1150 5100 1150
+$Comp
+L power:PWR_FLAG #FLG0102
+U 1 1 5D7279E3
+P 5500 6600
+F 0 "#FLG0102" H 5500 6675 50  0001 C CNN
+F 1 "PWR_FLAG" H 5500 6773 50  0000 C CNN
+F 2 "" H 5500 6600 50  0001 C CNN
+F 3 "~" H 5500 6600 50  0001 C CNN
+	1    5500 6600
+	-1   0    0    1
+$EndComp
+Wire Wire Line
+	5500 6600 5500 6350
+Wire Bus Line
+	4500 1550 4500 3000
+Wire Bus Line
+	7650 1550 7650 6050
+Connection ~ 5500 6350
+Wire Wire Line
+	5500 6350 5100 6350
 $EndSCHEMATC
