File: Hardware/DomesdayDuplicator-base-DE0Nano/de0-nano.sch (KiCad schematic (older format))
At the start: 3 parts

Commit message: Fixes to module and base - added component mapping to base and verified mirrored headers
Parts:
- gave numbers to parts that had none: 3
Connections:
- removed net +3V3: J201.29 (VCC3P3), J202.29 (VCC3P3), J203.1 (VCC3P3)
- no-connect marks 16 -> 19
Changed lines of the file:
@@
 $Descr A4 11693 8268
 encoding utf-8
-Sheet 2 5
+Sheet 2 6
 Title "Domesday Duplicator Base - DE0-Nano/FX3"
 Date "2019-09-02"
@@
 $EndDescr
 $Comp
-L DE0-Nano-Headers:GPIO-0 J?
+L DE0-Nano-Headers:GPIO-0 J201
 U 1 1 5D7279C0
 P 3450 2600
-F 0 "J?" H 3450 3815 50  0000 C CNN
+F 0 "J201" H 3450 3815 50  0000 C CNN
 F 1 "GPIO-0" H 3450 3724 50  0000 C CNN
 F 2 "Connector_PinSocket_2.54mm:PinSocket_2x20_P2.54mm_Vertical" H 3450 1500 50  0001 C CNN
@@
 $EndComp
 $Comp
-L DE0-Nano-Headers:GPIO-1 J?
+L DE0-Nano-Headers:GPIO-1 J202
 U 1 1 5D729381
 P 3450 5400
-F 0 "J?" H 3450 6615 50  0000 C CNN
+F 0 "J202" H 3450 6615 50  0000 C CNN
 F 1 "GPIO-1" H 3450 6524 50  0000 C CNN
 F 2 "Connector_PinSocket_2.54mm:PinSocket_2x20_P2.54mm_Vertical" H 3450 4300 50  0001 C CNN
@@
 $EndComp
 $Comp
-L DE0-Nano-Headers:GPIO-2 J?
+L DE0-Nano-Headers:GPIO-2 J203
 U 1 1 5D72B839
 P 8300 4200
-F 0 "J?" H 8300 5065 50  0000 C CNN
+F 0 "J203" H 8300 5065 50  0000 C CNN
 F 1 "GPIO-2" H 8300 4974 50  0000 C CNN
 F 2 "Connector_IDC:IDC-Header_2x13_P2.54mm_Vertical" H 8300 3450 50  0001 C CNN
@@
 	4650 2150 4650 3050
 $Comp
-L power:GND #PWR?
+L power:GND #PWR0203
 U 1 1 5D9000FE
 P 4650 6400
-F 0 "#PWR?" H 4650 6150 50  0001 C CNN
+F 0 "#PWR0203" H 4650 6150 50  0001 C CNN
 F 1 "GND" H 4655 6227 50  0000 C CNN
 F 2 "" H 4650 6400 50  0001 C CNN
@@
 	2250 4950 2250 4450
 Wire Wire Line
-	2850 5850 1950 5850
-Wire Wire Line
-	1950 5850 1950 4450
-Wire Wire Line
 	2850 2150 2250 2150
 Wire Wire Line
 	2250 2150 2250 1650
-Wire Wire Line
-	2850 3050 1950 3050
-Wire Wire Line
-	1950 3050 1950 1650
 $Comp
-L power:+5V #PWR?
+L power:+5V #PWR0201
 U 1 1 5D932AA7
 P 2250 1650
-F 0 "#PWR?" H 2250 1500 50  0001 C CNN
+F 0 "#PWR0201" H 2250 1500 50  0001 C CNN
 F 1 "+5V" H 2265 1823 50  0000 C CNN
 F 2 "" H 2250 1650 50  0001 C CNN
@@
 $EndComp
 $Comp
-L power:+5V #PWR?
+L power:+5V #PWR0202
 U 1 1 5D932D5F
 P 2250 4450
-F 0 "#PWR?" H 2250 4300 50  0001 C CNN
+F 0 "#PWR0202" H 2250 4300 50  0001 C CNN
 F 1 "+5V" H 2265 4623 50  0000 C CNN
 F 2 "" H 2250 4450 50  0001 C CNN
@@
 $EndComp
 $Comp
-L power:+3V3 #PWR?
-U 1 1 5D932F49
-P 1950 4450
-F 0 "#PWR?" H 1950 4300 50  0001 C CNN
-F 1 "+3V3" H 1965 4623 50  0000 C CNN
-F 2 "" H 1950 4450 50  0001 C CNN
-F 3 "" H 1950 4450 50  0001 C CNN
-	1    1950 4450
-	1    0    0    -1
-$EndComp
-$Comp
-L power:+3V3 #PWR?
-U 1 1 5D933122
-P 1950 1650
-F 0 "#PWR?" H 1950 1500 50  0001 C CNN
-F 1 "+3V3" H 1965 1823 50  0000 C CNN
-F 2 "" H 1950 1650 50  0001 C CNN
-F 3 "" H 1950 1650 50  0001 C CNN
-	1    1950 1650
-	1    0    0    -1
-$EndComp
-$Comp
-L power:+3V3 #PWR?
-U 1 1 5D933C17
-P 7550 3400
-F 0 "#PWR?" H 7550 3250 50  0001 C CNN
-F 1 "+3V3" H 7565 3573 50  0000 C CNN
-F 2 "" H 7550 3400 50  0001 C CNN
-F 3 "" H 7550 3400 50  0001 C CNN
-	1    7550 3400
-	1    0    0    -1
-$EndComp
-$Comp
-L power:GND #PWR?
+L power:GND #PWR0204
 U 1 1 5D934C93
 P 9050 4950
-F 0 "#PWR?" H 9050 4700 50  0001 C CNN
+F 0 "#PWR0204" H 9050 4700 50  0001 C CNN
 F 1 "GND" H 9055 4777 50  0000 C CNN
 F 2 "" H 9050 4950 50  0001 C CNN
@@
 Wire Wire Line
 	9050 4800 9050 4950
-Wire Wire Line
-	7650 3600 7550 3600
-Wire Wire Line
-	7550 3600 7550 3400
 NoConn ~ 8950 3600
 NoConn ~ 8950 3700
@@
 Text HLabel 5500 6650 2    50   BiDi ~ 0
 MOD1_D[0..15]
+NoConn ~ 2850 5850
+NoConn ~ 2850 3050
+NoConn ~ 7650 3600
 Wire Bus Line
 	7050 3000 7050 4300

Commit message: Mechanical set up of base board and basic routing
Parts:
- J203: footprint Connector_IDC:IDC-Header_2x13_P2.54mm_Vertical -> Connector_IDC:IDC-Header_2x13_P2.54mm_Horizontal
Connections:
- net MOD0_CLK: now also J201.22 (GPIO_0_17); no longer J202.21 (GPIO_1_16)
- net MOD0_D0: now also J201.40 (GPIO_0_33); no longer J202.2 (GPIO_1_0)
- net MOD0_D1: now also J201.39 (GPIO_0_32); no longer J202.4 (GPIO_1_1)
- net MOD0_D10: now also J201.28 (GPIO_0_23); no longer J202.15 (GPIO_1_10)
- net MOD0_D11: now also J201.27 (GPIO_0_22); no longer J202.16 (GPIO_1_11)
- net MOD0_D12: now also J201.26 (GPIO_0_21); no longer J202.17 (GPIO_1_12)
- net MOD0_D13: now also J201.25 (GPIO_0_20); no longer J202.18 (GPIO_1_13)
- net MOD0_D14: now also J201.24 (GPIO_0_19); no longer J202.19 (GPIO_1_14)
- net MOD0_D15: now also J201.23 (GPIO_0_18); no longer J202.20 (GPIO_1_15)
- net MOD0_D2: now also J201.38 (GPIO_0_31); no longer J202.5 (GPIO_1_2)
- net MOD0_D3: now also J201.37 (GPIO_0_30); no longer J202.6 (GPIO_1_3)
- net MOD0_D4: now also J201.36 (GPIO_0_29); no longer J202.7 (GPIO_1_4)
- net MOD0_D5: now also J201.35 (GPIO_0_28); no longer J202.8 (GPIO_1_5)
- net MOD0_D6: now also J201.34 (GPIO_0_27); no longer J202.9 (GPIO_1_6)
- net MOD0_D7: now also J201.33 (GPIO_0_26); no longer J202.10 (GPIO_1_7)
- net MOD0_D8: now also J201.32 (GPIO_0_25); no longer J202.13 (GPIO_1_8)
- net MOD0_D9: now also J201.31 (GPIO_0_24); no longer J202.14 (GPIO_1_9)
- net MOD1_CLK: now also J201.2 (GPIO_0_0); no longer J202.40 (GPIO_1_33)
- net MOD1_D0: now also J201.21 (GPIO_0_16); no longer J202.22 (GPIO_1_17)
- net MOD1_D1: now also J201.20 (GPIO_0_15); no longer J202.23 (GPIO_1_18)
- net MOD1_D10: now also J201.9 (GPIO_0_6); no longer J202.34 (GPIO_1_27)
- net MOD1_D11: now also J201.8 (GPIO_0_5); no longer J202.35 (GPIO_1_28)
- net MOD1_D12: now also J201.7 (GPIO_0_4); no longer J202.36 (GPIO_1_29)
- net MOD1_D13: now also J201.6 (GPIO_0_3); no longer J202.37 (GPIO_1_30)
- net MOD1_D14: now also J201.5 (GPIO_0_2); no longer J202.38 (GPIO_1_31)
- net MOD1_D15: now also J201.4 (GPIO_0_1); no longer J202.39 (GPIO_1_32)
- net MOD1_D2: now also J201.19 (GPIO_0_14); no longer J202.24 (GPIO_1_19)
- net MOD1_D3: now also J201.18 (GPIO_0_13); no longer J202.25 (GPIO_1_20)
- net MOD1_D4: now also J201.17 (GPIO_0_12); no longer J202.26 (GPIO_1_21)
- net MOD1_D5: now also J201.16 (GPIO_0_11); no longer J202.27 (GPIO_1_22)
- net MOD1_D6: now also J201.15 (GPIO_0_10); no longer J202.28 (GPIO_1_23)
- net MOD1_D7: now also J201.14 (GPIO_0_9); no longer J202.31 (GPIO_1_24)
- net MOD1_D8: now also J201.13 (GPIO_0_8); no longer J202.32 (GPIO_1_25)
- net MOD1_D9: now also J201.10 (GPIO_0_7); no longer J202.33 (GPIO_1_26)
- net USB_CTL0: now also J203.17 (GPIO-2-12); no longer J203.5 (GPIO-2-0)
- net USB_CTL1: now also J203.16 (GPIO-2-11); no longer J203.6 (GPIO-2-1)
- net USB_CTL10: now also J203.7 (GPIO-2-2); no longer J203.15 (GPIO-2-10)
- net USB_CTL11: now also J203.6 (GPIO-2-1); no longer J203.16 (GPIO-2-11)
- net USB_CTL12: now also J203.5 (GPIO-2-0); no longer J203.17 (GPIO-2-12)
- net USB_CTL2: now also J203.15 (GPIO-2-10); no longer J203.7 (GPIO-2-2)
- net USB_CTL3: now also J203.14 (GPIO-2-9); no longer J203.8 (GPIO-2-3)
- net USB_CTL4: now also J203.13 (GPIO-2-8); no longer J203.9 (GPIO-2-4)
- net USB_CTL5: now also J203.12 (GPIO-2-7); no longer J203.10 (GPIO-2-5)
- net USB_CTL7: now also J203.10 (GPIO-2-5); no longer J203.12 (GPIO-2-7)
- net USB_CTL8: now also J203.9 (GPIO-2-4); no longer J203.13 (GPIO-2-8)
- net USB_CTL9: now also J203.8 (GPIO-2-3); no longer J203.14 (GPIO-2-9)
- net USB_DATA0: now also J202.5 (GPIO_1_2); no longer J201.2 (GPIO_0_0)
- net USB_DATA1: now also J202.6 (GPIO_1_3); no longer J201.4 (GPIO_0_1)
- net USB_DATA10: now also J202.25 (GPIO_1_20); no longer J201.15 (GPIO_0_10)
- net USB_DATA11: now also J202.27 (GPIO_1_22); no longer J201.16 (GPIO_0_11)
- net USB_DATA12: now also J202.31 (GPIO_1_24); no longer J201.17 (GPIO_0_12)
- net USB_DATA13: now also J202.33 (GPIO_1_26); no longer J201.18 (GPIO_0_13)
- net USB_DATA14: now also J202.35 (GPIO_1_28); no longer J201.19 (GPIO_0_14)
- net USB_DATA15: now also J202.37 (GPIO_1_30); no longer J201.20 (GPIO_0_15)
- net USB_DATA16: now also J202.2 (GPIO_1_0); no longer J201.21 (GPIO_0_16)
- net USB_DATA17: now also J202.4 (GPIO_1_1); no longer J201.22 (GPIO_0_17)
- net USB_DATA18: now also J202.10 (GPIO_1_7); no longer J201.23 (GPIO_0_18)
- net USB_DATA19: now also J202.14 (GPIO_1_9); no longer J201.24 (GPIO_0_19)
- net USB_DATA2: now also J202.7 (GPIO_1_4); no longer J201.5 (GPIO_0_2)
- net USB_DATA20: now also J202.16 (GPIO_1_11); no longer J201.25 (GPIO_0_20)
- net USB_DATA21: now also J202.18 (GPIO_1_13); no longer J201.26 (GPIO_0_21)
- net USB_DATA22: now also J202.20 (GPIO_1_15); no longer J201.27 (GPIO_0_22)
- net USB_DATA23: now also J202.22 (GPIO_1_17); no longer J201.28 (GPIO_0_23)
- net USB_DATA24: now also J202.24 (GPIO_1_19); no longer J201.31 (GPIO_0_24)
- net USB_DATA25: now also J202.26 (GPIO_1_21); no longer J201.32 (GPIO_0_25)
- net USB_DATA26: now also J202.28 (GPIO_1_23); no longer J201.33 (GPIO_0_26)
- net USB_DATA27: now also J202.32 (GPIO_1_25); no longer J201.34 (GPIO_0_27)
- net USB_DATA28: now also J202.34 (GPIO_1_27); no longer J201.35 (GPIO_0_28)
- net USB_DATA29: now also J202.36 (GPIO_1_29); no longer J201.36 (GPIO_0_29)
- net USB_DATA3: now also J202.9 (GPIO_1_6); no longer J201.6 (GPIO_0_3)
- net USB_DATA30: now also J202.38 (GPIO_1_31); no longer J201.37 (GPIO_0_30)
- net USB_DATA31: now also J202.40 (GPIO_1_33); no longer J201.38 (GPIO_0_31)
- net USB_DATA4: now also J202.13 (GPIO_1_8); no longer J201.7 (GPIO_0_4)
- net USB_DATA5: now also J202.15 (GPIO_1_10); no longer J201.8 (GPIO_0_5)
- net USB_DATA6: now also J202.17 (GPIO_1_12); no longer J201.9 (GPIO_0_6)
- net USB_DATA7: now also J202.19 (GPIO_1_14); no longer J201.10 (GPIO_0_7)
- net USB_DATA8: now also J202.21 (GPIO_1_16); no longer J201.13 (GPIO_0_8)
- net USB_DATA9: now also J202.23 (GPIO_1_18); no longer J201.14 (GPIO_0_9)
- net USB_PCLK: now also J202.8 (GPIO_1_5); no longer J201.39 (GPIO_0_32)
Other:
- note added: "0 to 15 on this side\n"
- note added: "16-30 on this side\n"
- moved on the sheet: J201, J202
