File: Hardware/DomesdayDuplicator-base-DE0Nano/power-supply.sch (KiCad schematic (older format))
At the start: 6 parts

Commit message: Fixes to module and base - added component mapping to base and verified mirrored headers
Parts:
- C501, C504: renamed from C?; footprint (none) -> Capacitor_SMD:C_0805_2012Metric
- C502, C503: renamed from C?; footprint (none) -> Capacitor_Tantalum_SMD:CP_EIA-3528-21_Kemet-B
- L501: renamed from L?; footprint (none) -> Inductor_SMD:L_Bourns_SRN8040TA
- U501: renamed from U?; footprint (none) -> Package_TO_SOT_SMD:SOT-223-3_TabPin2
Changed lines of the file:
@@
 $Descr A4 11693 8268
 encoding utf-8
-Sheet 5 5
+Sheet 5 6
 Title "Domesday Duplicator Base - DE0-Nano/FX3"
 Date "2019-09-02"
@@
 $EndDescr
 $Comp
-L Regulator_Linear:LM1117-3.3 U?
+L Regulator_Linear:LM1117-3.3 U501
 U 1 1 5D780D1E
 P 6200 3800
-F 0 "U?" H 6200 4042 50  0000 C CNN
+F 0 "U501" H 6200 4042 50  0000 C CNN
 F 1 "LM1117-3.3" H 6200 3951 50  0000 C CNN
-F 2 "" H 6200 3800 50  0001 C CNN
+F 2 "Package_TO_SOT_SMD:SOT-223-3_TabPin2" H 6200 3800 50  0001 C CNN
 F 3 "http://www.ti.com/lit/ds/symlink/lm1117.pdf" H 6200 3800 50  0001 C CNN
 	1    6200 3800
@@
 $EndComp
 $Comp
-L Device:C C?
+L Device:C C501
 U 1 1 5D781507
 P 4800 4050
-F 0 "C?" H 4915 4096 50  0000 L CNN
+F 0 "C501" H 4915 4096 50  0000 L CNN
 F 1 "100nF" H 4915 4005 50  0000 L CNN
-F 2 "" H 4838 3900 50  0001 C CNN
+F 2 "Capacitor_SMD:C_0805_2012Metric" H 4838 3900 50  0001 C CNN
 F 3 "~" H 4800 4050 50  0001 C CNN
 	1    4800 4050
@@
 $EndComp
 $Comp
-L Device:C C?
+L Device:C C504
 U 1 1 5D7825F0
 P 7550 4050
-F 0 "C?" H 7665 4096 50  0000 L CNN
+F 0 "C504" H 7665 4096 50  0000 L CNN
 F 1 "100nF" H 7665 4005 50  0000 L CNN
-F 2 "" H 7588 3900 50  0001 C CNN
+F 2 "Capacitor_SMD:C_0805_2012Metric" H 7588 3900 50  0001 C CNN
 F 3 "~" H 7550 4050 50  0001 C CNN
 	1    7550 4050
@@
 $EndComp
 $Comp
-L Device:CP C?
+L Device:CP C502
 U 1 1 5D7828A4
 P 5450 4050
-F 0 "C?" H 5568 4096 50  0000 L CNN
+F 0 "C502" H 5568 4096 50  0000 L CNN
 F 1 "10uF tant" H 5568 4005 50  0000 L CNN
-F 2 "" H 5488 3900 50  0001 C CNN
+F 2 "Capacitor_Tantalum_SMD:CP_EIA-3528-21_Kemet-B" H 5488 3900 50  0001 C CNN
 F 3 "~" H 5450 4050 50  0001 C CNN
 	1    5450 4050
@@
 $EndComp
 $Comp
-L Device:CP C?
+L Device:CP C503
 U 1 1 5D783926
 P 6950 4050
-F 0 "C?" H 7068 4096 50  0000 L CNN
+F 0 "C503" H 7068 4096 50  0000 L CNN
 F 1 "10uF tant" H 7068 4005 50  0000 L CNN
-F 2 "" H 6988 3900 50  0001 C CNN
+F 2 "Capacitor_Tantalum_SMD:CP_EIA-3528-21_Kemet-B" H 6988 3900 50  0001 C CNN
 F 3 "~" H 6950 4050 50  0001 C CNN
 	1    6950 4050
@@
 	6950 3800 6950 3900
 Wire Wire Line
-	5450 3800 4800 3800
+	5450 3800 5200 3800
 Wire Wire Line
 	4800 3800 4800 3900
@@
 	6950 4300 7550 4300
 $Comp
-L power:GND #PWR?
+L power:GND #PWR0503
 U 1 1 5D78D444
 P 6200 4400
-F 0 "#PWR?" H 6200 4150 50  0001 C CNN
+F 0 "#PWR0503" H 6200 4150 50  0001 C CNN
 F 1 "GND" H 6205 4227 50  0000 C CNN
 F 2 "" H 6200 4400 50  0001 C CNN
@@
 	6200 4400 6200 4300
 $Comp
-L power:+3.3VA #PWR?
+L power:+3.3VA #PWR0504
 U 1 1 5D78D771
 P 7550 3700
-F 0 "#PWR?" H 7550 3550 50  0001 C CNN
+F 0 "#PWR0504" H 7550 3550 50  0001 C CNN
 F 1 "+3.3VA" H 7565 3873 50  0000 C CNN
 F 2 "" H 7550 3700 50  0001 C CNN
@@
 $EndComp
 $Comp
-L power:+5VA #PWR?
+L power:+5VA #PWR0502
 U 1 1 5D78D8CF
 P 4800 3700
-F 0 "#PWR?" H 4800 3550 50  0001 C CNN
+F 0 "#PWR0502" H 4800 3550 50  0001 C CNN
 F 1 "+5VA" H 4815 3873 50  0000 C CNN
 F 2 "" H 4800 3700 50  0001 C CNN
@@
 $EndComp
 $Comp
-L Device:L L?
+L Device:L L501
 U 1 1 5D78DAC6
 P 4350 3800
-F 0 "L?" V 4540 3800 50  0000 C CNN
+F 0 "L501" V 4540 3800 50  0000 C CNN
 F 1 "100uH" V 4449 3800 50  0000 C CNN
-F 2 "" H 4350 3800 50  0001 C CNN
+F 2 "Inductor_SMD:L_Bourns_SRN8040TA" H 4350 3800 50  0001 C CNN
 F 3 "~" H 4350 3800 50  0001 C CNN
 	1    4350 3800
@@
 $EndComp
 $Comp
-L power:+5V #PWR?
+L power:+5V #PWR0501
 U 1 1 5D78E235
 P 3950 3700
-F 0 "#PWR?" H 3950 3550 50  0001 C CNN
+F 0 "#PWR0501" H 3950 3550 50  0001 C CNN
 F 1 "+5V" H 3965 3873 50  0000 C CNN
 F 2 "" H 3950 3700 50  0001 C CNN
@@
 	7550 3800 7550 3700
 Connection ~ 7550 3800
+$Comp
+L power:PWR_FLAG #FLG0103
+U 1 1 5D72C85F
+P 5200 3700
+F 0 "#FLG0103" H 5200 3775 50  0001 C CNN
+F 1 "PWR_FLAG" H 5200 3873 50  0000 C CNN
+F 2 "" H 5200 3700 50  0001 C CNN
+F 3 "~" H 5200 3700 50  0001 C CNN
+	1    5200 3700
+	1    0    0    -1
+$EndComp
+Wire Wire Line
+	5200 3700 5200 3800
+Connection ~ 5200 3800
+Wire Wire Line
+	5200 3800 4800 3800
 $EndSCHEMATC
