File: Hardware/DomesdayDuplicator-base-DE0Nano/DomesdayDuplicator-base-DE0Nano.kicad_pcb (KiCad board)
At the start: 2 copper layers, 30 parts, among them J201 GPIO-0, J202 GPIO-1, J203 GPIO-2, J301 GPIFII_J6, J302 GPIFII_J7, J401 MOD0 Back, J402 MOD1 Back, J403 MOD0 Front, J404 MOD1 Front, U501 LM1117-3.3

Commit message: Work on the ADS825 module to determine the overall module dimensions and mounting
Parts:
- added RN401: 22R, Resistor_SMD:R_Array_Convex_4x1206, F.Cu at (62.6, 140.3)
- added RN402: 22R, Resistor_SMD:R_Array_Convex_4x1206, F.Cu at (68.0, 140.3)
- added RN403: 22R, Resistor_SMD:R_Array_Convex_4x1206, F.Cu at (62.6, 147.0)
- added RN404: 22R, Resistor_SMD:R_Array_Convex_4x1206, F.Cu at (68.0, 147.0)
- added RN405: 22R, Resistor_SMD:R_Array_Convex_4x1206, F.Cu at (73.5, 140.3)
- added RN406: 22R, Resistor_SMD:R_Array_Convex_4x1206, F.Cu at (78.9, 140.3)
- added RN407: 22R, Resistor_SMD:R_Array_Convex_4x1206, F.Cu at (73.5, 147.0)
- added RN408: 22R, Resistor_SMD:R_Array_Convex_4x1206, F.Cu at (78.9, 147.0)
- J401, J403, J404: footprint Connector_PinSocket_1.27mm:PinSocket_2x10_P1.27mm_Vertical_SMD -> Connector_Hirose:Hirose_DF12_DF12C3.0-20DS-0.5V_2x10_P0.50mm_Vertical
- J402: value MOD1 Back -> MOD0 Back; footprint Connector_PinSocket_1.27mm:PinSocket_2x10_P1.27mm_Vertical_SMD -> Connector_Hirose:Hirose_DF12_DF12C3.0-20DS-0.5V_2x10_P0.50mm_Vertical
- moved J402 45.9 mm to (56.0, 144.3)
Connections:
- J401 pad 1: /DE0-Nano/MOD0_D0 -> Net-(J401-Pad1)
- J401 pad 10: /DE0-Nano/MOD0_D9 -> Net-(J401-Pad10)
- J401 pad 11: /DE0-Nano/MOD0_D10 -> Net-(J401-Pad11)
- J401 pad 12: /DE0-Nano/MOD0_D11 -> Net-(J401-Pad12)
- J401 pad 13: /DE0-Nano/MOD0_D12 -> Net-(J401-Pad13)
- J401 pad 14: /DE0-Nano/MOD0_D13 -> Net-(J401-Pad14)
- J401 pad 15: /DE0-Nano/MOD0_D14 -> Net-(J401-Pad15)
- J401 pad 16: /DE0-Nano/MOD0_D15 -> Net-(J401-Pad16)
- J401 pad 2: /DE0-Nano/MOD0_D1 -> Net-(J401-Pad2)
- J401 pad 3: /DE0-Nano/MOD0_D2 -> Net-(J401-Pad3)
- J401 pad 4: /DE0-Nano/MOD0_D3 -> Net-(J401-Pad4)
- J401 pad 5: /DE0-Nano/MOD0_D4 -> Net-(J401-Pad5)
- J401 pad 6: /DE0-Nano/MOD0_D5 -> Net-(J401-Pad6)
- J401 pad 7: /DE0-Nano/MOD0_D6 -> Net-(J401-Pad7)
- J401 pad 8: /DE0-Nano/MOD0_D7 -> Net-(J401-Pad8)
- J401 pad 9: /DE0-Nano/MOD0_D8 -> Net-(J401-Pad9)
- J402 pad 1: /DE0-Nano/MOD1_D0 -> Net-(J402-Pad1)
- J402 pad 10: /DE0-Nano/MOD1_D9 -> Net-(J402-Pad10)
- J402 pad 11: /DE0-Nano/MOD1_D10 -> Net-(J402-Pad11)
- J402 pad 12: /DE0-Nano/MOD1_D11 -> Net-(J402-Pad12)
- J402 pad 13: /DE0-Nano/MOD1_D12 -> Net-(J402-Pad13)
- J402 pad 14: /DE0-Nano/MOD1_D13 -> Net-(J402-Pad14)
- J402 pad 15: /DE0-Nano/MOD1_D14 -> Net-(J402-Pad15)
- J402 pad 16: /DE0-Nano/MOD1_D15 -> Net-(J402-Pad16)
- J402 pad 2: /DE0-Nano/MOD1_D1 -> Net-(J402-Pad2)
- J402 pad 3: /DE0-Nano/MOD1_D2 -> Net-(J402-Pad3)
- J402 pad 4: /DE0-Nano/MOD1_D3 -> Net-(J402-Pad4)
- J402 pad 5: /DE0-Nano/MOD1_D4 -> Net-(J402-Pad5)
- J402 pad 6: /DE0-Nano/MOD1_D5 -> Net-(J402-Pad6)
- J402 pad 7: /DE0-Nano/MOD1_D6 -> Net-(J402-Pad7)
- J402 pad 8: /DE0-Nano/MOD1_D7 -> Net-(J402-Pad8)
- J402 pad 9: /DE0-Nano/MOD1_D8 -> Net-(J402-Pad9)

Commit message: Mechanical set up of base board and basic routing
Parts:
- removed J403: MOD0 Front, Connector_Hirose:Hirose_DF12_DF12C3.0-20DS-0.5V_2x10_P0.50mm_Vertical
- removed J404: MOD1 Front, Connector_Hirose:Hirose_DF12_DF12C3.0-20DS-0.5V_2x10_P0.50mm_Vertical
- removed the RN403 at (62.6, 147.0)
- removed the RN404 at (68.0, 147.0)
- added H604: MountingHole, MountingHole:MountingHole_3.2mm_M3, F.Cu at (199.6, 55.0)
- added H606: MountingHole, MountingHole:MountingHole_2.2mm_M2, F.Cu at (106.7, 122.6)
- added RN405: 22R, Resistor_SMD:R_Array_Convex_4x1206, F.Cu at (132.2, 98.2)
- added RN406: 22R, Resistor_SMD:R_Array_Convex_4x1206, F.Cu at (132.2, 104.8)
- C406: value 100nF -> 2.2uF tant; footprint Capacitor_SMD:C_0805_2012Metric -> Capacitor_Tantalum_SMD:CP_EIA-3216-18_Kemet-A
- C407: value 2.2uF tant -> 100nF; footprint Capacitor_Tantalum_SMD:CP_EIA-3216-18_Kemet-A -> Capacitor_SMD:C_0805_2012Metric
- H603: footprint MountingHole:MountingHole_3.2mm_M3 -> MountingHole:MountingHole_2.2mm_M2
- J201, J202: moved to B.Cu
- J203: footprint Connector_IDC:IDC-Header_2x13_P2.54mm_Vertical -> Connector_IDC:IDC-Header_2x13_P2.54mm_Horizontal
- J401: value MOD0 Back -> MOD0_Connector; footprint Connector_Hirose:Hirose_DF12_DF12C3.0-20DS-0.5V_2x10_P0.50mm_Vertical -> Connector_IDC:IDC-Header_2x10_P2.54mm_Vertical
- J402: value MOD0 Back -> MOD1_Connector; footprint Connector_Hirose:Hirose_DF12_DF12C3.0-20DS-0.5V_2x10_P0.50mm_Vertical -> Connector_IDC:IDC-Header_2x10_P2.54mm_Vertical
- moved FID601 110.3 mm to (115.8, 56.0)
- moved H601 108.4 mm to (107.7, 55.0)
- moved H603 102.1 mm to (106.7, 83.2)
- moved FID603 97.8 mm to (115.8, 138.3)
- moved RN401 97.3 mm to (132.2, 72.4)
- moved J402 89.5 mm to (139.1, 111.1)
- moved RN402 88.9 mm to (132.2, 78.7)
- moved H602 86.2 mm to (107.7, 138.8)
- moved RN403 80.6 mm to (132.2, 85.1)
- moved J301 76.5 mm to (154.9, 125.6), turned to 180 degrees
- moved J401 73.5 mm to (139.1, 71.8)
- moved RN404 72.3 mm to (132.2, 91.4)
- moved C405 69.9 mm to (146.3, 93.6), turned to 270 degrees
- moved J202 69.3 mm to (167.8, 70.5), turned to 180 degrees
- moved C402 67.1 mm to (148.8, 98.7), turned to 90 degrees
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- renumbered C403 to C402, C402 to C403, H604 to H605, RN405 to RN403, RN406 to RN404
Connections:
- net Net-(J401-Pad1) renamed /Module Headers/M0_D0
- J201 pad 10: /Cypress FX3/USB_DATA7 -> /DE0-Nano/MOD1_D9
- J201 pad 13: /Cypress FX3/USB_DATA8 -> /DE0-Nano/MOD1_D8
- J201 pad 14: /Cypress FX3/USB_DATA9 -> /DE0-Nano/MOD1_D7
- J201 pad 15: /Cypress FX3/USB_DATA10 -> /DE0-Nano/MOD1_D6
- J201 pad 16: /Cypress FX3/USB_DATA11 -> /DE0-Nano/MOD1_D5
- J201 pad 17: /Cypress FX3/USB_DATA12 -> /DE0-Nano/MOD1_D4
- J201 pad 18: /Cypress FX3/USB_DATA13 -> /DE0-Nano/MOD1_D3
- J201 pad 19: /Cypress FX3/USB_DATA14 -> /DE0-Nano/MOD1_D2
- J201 pad 2: /Cypress FX3/USB_DATA0 -> /DE0-Nano/MOD1_CLK
- J201 pad 20: /Cypress FX3/USB_DATA15 -> /DE0-Nano/MOD1_D1
- J201 pad 21: /Cypress FX3/USB_DATA16 -> /DE0-Nano/MOD1_D0
- J201 pad 22: /Cypress FX3/USB_DATA17 -> /DE0-Nano/MOD0_CLK
- J201 pad 23: /Cypress FX3/USB_DATA18 -> /DE0-Nano/MOD0_D15
- J201 pad 24: /Cypress FX3/USB_DATA19 -> /DE0-Nano/MOD0_D14
- J201 pad 25: /Cypress FX3/USB_DATA20 -> /DE0-Nano/MOD0_D13
- J201 pad 26: /Cypress FX3/USB_DATA21 -> /DE0-Nano/MOD0_D12
- J201 pad 27: /Cypress FX3/USB_DATA22 -> /DE0-Nano/MOD0_D11
- J201 pad 28: /Cypress FX3/USB_DATA23 -> /DE0-Nano/MOD0_D10
- J201 pad 31: /Cypress FX3/USB_DATA24 -> /DE0-Nano/MOD0_D9
- J201 pad 32: /Cypress FX3/USB_DATA25 -> /DE0-Nano/MOD0_D8
- J201 pad 33: /Cypress FX3/USB_DATA26 -> /DE0-Nano/MOD0_D7
- J201 pad 34: /Cypress FX3/USB_DATA27 -> /DE0-Nano/MOD0_D6
- J201 pad 35: /Cypress FX3/USB_DATA28 -> /DE0-Nano/MOD0_D5
- J201 pad 36: /Cypress FX3/USB_DATA29 -> /DE0-Nano/MOD0_D4
- J201 pad 37: /Cypress FX3/USB_DATA30 -> /DE0-Nano/MOD0_D3
- J201 pad 38: /Cypress FX3/USB_DATA31 -> /DE0-Nano/MOD0_D2
- J201 pad 39: /Cypress FX3/USB_PCLK -> /DE0-Nano/MOD0_D1
- J201 pad 4: /Cypress FX3/USB_DATA1 -> /DE0-Nano/MOD1_D15
- J201 pad 40: (no net) -> /DE0-Nano/MOD0_D0
- J201 pad 5: /Cypress FX3/USB_DATA2 -> /DE0-Nano/MOD1_D14
- J201 pad 6: /Cypress FX3/USB_DATA3 -> /DE0-Nano/MOD1_D13
- J201 pad 7: /Cypress FX3/USB_DATA4 -> /DE0-Nano/MOD1_D12
- J201 pad 8: /Cypress FX3/USB_DATA5 -> /DE0-Nano/MOD1_D11
- J201 pad 9: /Cypress FX3/USB_DATA6 -> /DE0-Nano/MOD1_D10
- J202 pad 10: /DE0-Nano/MOD0_D7 -> /Cypress FX3/USB_DATA18
- J202 pad 13: /DE0-Nano/MOD0_D8 -> /Cypress FX3/USB_DATA4
- J202 pad 14: /DE0-Nano/MOD0_D9 -> /Cypress FX3/USB_DATA19
- J202 pad 15: /DE0-Nano/MOD0_D10 -> /Cypress FX3/USB_DATA5
- J202 pad 16: /DE0-Nano/MOD0_D11 -> /Cypress FX3/USB_DATA20
- J202 pad 17: /DE0-Nano/MOD0_D12 -> /Cypress FX3/USB_DATA6
- J202 pad 18: /DE0-Nano/MOD0_D13 -> /Cypress FX3/USB_DATA21
- J202 pad 19: /DE0-Nano/MOD0_D14 -> /Cypress FX3/USB_DATA7
- J202 pad 2: /DE0-Nano/MOD0_D0 -> /Cypress FX3/USB_DATA16
- J202 pad 20: /DE0-Nano/MOD0_D15 -> /Cypress FX3/USB_DATA22
- J202 pad 21: /DE0-Nano/MOD0_CLK -> /Cypress FX3/USB_DATA8
- J202 pad 22: /DE0-Nano/MOD1_D0 -> /Cypress FX3/USB_DATA23
- J202 pad 23: /DE0-Nano/MOD1_D1 -> /Cypress FX3/USB_DATA9
- J202 pad 24: /DE0-Nano/MOD1_D2 -> /Cypress FX3/USB_DATA24
- J202 pad 25: /DE0-Nano/MOD1_D3 -> /Cypress FX3/USB_DATA10
- J202 pad 26: /DE0-Nano/MOD1_D4 -> /Cypress FX3/USB_DATA25
- J202 pad 27: /DE0-Nano/MOD1_D5 -> /Cypress FX3/USB_DATA11
- J202 pad 28: /DE0-Nano/MOD1_D6 -> /Cypress FX3/USB_DATA26
- J202 pad 31: /DE0-Nano/MOD1_D7 -> /Cypress FX3/USB_DATA12
- J202 pad 32: /DE0-Nano/MOD1_D8 -> /Cypress FX3/USB_DATA27
- J202 pad 33: /DE0-Nano/MOD1_D9 -> /Cypress FX3/USB_DATA13
- J202 pad 34: /DE0-Nano/MOD1_D10 -> /Cypress FX3/USB_DATA28
- J202 pad 35: /DE0-Nano/MOD1_D11 -> /Cypress FX3/USB_DATA14
- J202 pad 36: /DE0-Nano/MOD1_D12 -> /Cypress FX3/USB_DATA29
- J202 pad 37: /DE0-Nano/MOD1_D13 -> /Cypress FX3/USB_DATA15
- J202 pad 38: /DE0-Nano/MOD1_D14 -> /Cypress FX3/USB_DATA30
- J202 pad 39: /DE0-Nano/MOD1_D15 -> (no net)
- J202 pad 4: /DE0-Nano/MOD0_D1 -> /Cypress FX3/USB_DATA17
- J202 pad 40: /DE0-Nano/MOD1_CLK -> /Cypress FX3/USB_DATA31
- J202 pad 5: /DE0-Nano/MOD0_D2 -> /Cypress FX3/USB_DATA0
- J202 pad 6: /DE0-Nano/MOD0_D3 -> /Cypress FX3/USB_DATA1
- J202 pad 7: /DE0-Nano/MOD0_D4 -> /Cypress FX3/USB_DATA2
- J202 pad 8: /DE0-Nano/MOD0_D5 -> /Cypress FX3/USB_PCLK
- J202 pad 9: /DE0-Nano/MOD0_D6 -> /Cypress FX3/USB_DATA3
- J203 pad 10: /Cypress FX3/USB_CTL5 -> /Cypress FX3/USB_CTL7
- J203 pad 12: /Cypress FX3/USB_CTL7 -> /Cypress FX3/USB_CTL5
- J203 pad 13: /Cypress FX3/USB_CTL8 -> /Cypress FX3/USB_CTL4
- J203 pad 14: /Cypress FX3/USB_CTL9 -> /Cypress FX3/USB_CTL3
- J203 pad 15: /Cypress FX3/USB_CTL10 -> /Cypress FX3/USB_CTL2
- J203 pad 16: /Cypress FX3/USB_CTL11 -> /Cypress FX3/USB_CTL1
- J203 pad 17: /Cypress FX3/USB_CTL12 -> /Cypress FX3/USB_CTL0
- J203 pad 5: /Cypress FX3/USB_CTL0 -> /Cypress FX3/USB_CTL12
- J203 pad 6: /Cypress FX3/USB_CTL1 -> /Cypress FX3/USB_CTL11
- J203 pad 7: /Cypress FX3/USB_CTL2 -> /Cypress FX3/USB_CTL10
- J203 pad 8: /Cypress FX3/USB_CTL3 -> /Cypress FX3/USB_CTL9
- J203 pad 9: /Cypress FX3/USB_CTL4 -> /Cypress FX3/USB_CTL8
- J401 pad 10: Net-(J401-Pad10) -> /Module Headers/M0_D9
- J401 pad 11: Net-(J401-Pad11) -> /Module Headers/M0_D10
- J401 pad 12: Net-(J401-Pad12) -> /Module Headers/M0_D11
- J401 pad 13: Net-(J401-Pad13) -> /Module Headers/M0_D12
- J401 pad 14: Net-(J401-Pad14) -> /Module Headers/M0_D13
- J401 pad 15: Net-(J401-Pad15) -> /Module Headers/M0_D14
- J401 pad 16: Net-(J401-Pad16) -> /Module Headers/M0_D15
- J401 pad 2: Net-(J401-Pad2) -> /Module Headers/M0_D1
- J401 pad 3: Net-(J401-Pad3) -> /Module Headers/M0_D2
- J401 pad 4: Net-(J401-Pad4) -> /Module Headers/M0_D3
- J401 pad 5: Net-(J401-Pad5) -> /Module Headers/M0_D4
- J401 pad 6: Net-(J401-Pad6) -> /Module Headers/M0_D5
- J401 pad 7: Net-(J401-Pad7) -> /Module Headers/M0_D6
- J401 pad 8: Net-(J401-Pad8) -> /Module Headers/M0_D7
- J401 pad 9: Net-(J401-Pad9) -> /Module Headers/M0_D8
- J402 pad 1: Net-(J402-Pad1) -> /Module Headers/M1_D0
- J402 pad 10: Net-(J402-Pad10) -> /Module Headers/M1_D9
- J402 pad 11: Net-(J402-Pad11) -> /Module Headers/M1_D10
- J402 pad 12: Net-(J402-Pad12) -> /Module Headers/M1_D11
- J402 pad 13: Net-(J402-Pad13) -> /Module Headers/M1_D12
- J402 pad 14: Net-(J402-Pad14) -> /Module Headers/M1_D13
- J402 pad 15: Net-(J402-Pad15) -> /Module Headers/M1_D14
- J402 pad 16: Net-(J402-Pad16) -> /Module Headers/M1_D15
- J402 pad 2: Net-(J402-Pad2) -> /Module Headers/M1_D1
- J402 pad 3: Net-(J402-Pad3) -> /Module Headers/M1_D2
- J402 pad 4: Net-(J402-Pad4) -> /Module Headers/M1_D3
- J402 pad 5: Net-(J402-Pad5) -> /Module Headers/M1_D4
- J402 pad 6: Net-(J402-Pad6) -> /Module Headers/M1_D5
- J402 pad 7: Net-(J402-Pad7) -> /Module Headers/M1_D6
- J402 pad 8: Net-(J402-Pad8) -> /Module Headers/M1_D7
- J402 pad 9: Net-(J402-Pad9) -> /Module Headers/M1_D8
- RN401 pad 2: /DE0-Nano/MOD0_D2 -> /DE0-Nano/MOD0_D1
- RN401 pad 3: /DE0-Nano/MOD0_D4 -> /DE0-Nano/MOD0_D2
- RN401 pad 4: /DE0-Nano/MOD0_D6 -> /DE0-Nano/MOD0_D3
- RN401 pad 5: Net-(J401-Pad7) -> /Module Headers/M0_D3
- RN401 pad 6: Net-(J401-Pad5) -> /Module Headers/M0_D2
- RN401 pad 7: Net-(J401-Pad3) -> /Module Headers/M0_D1
- RN402 pad 1: /DE0-Nano/MOD0_D8 -> /DE0-Nano/MOD0_D4
- RN402 pad 2: /DE0-Nano/MOD0_D10 -> /DE0-Nano/MOD0_D5
- RN402 pad 3: /DE0-Nano/MOD0_D12 -> /DE0-Nano/MOD0_D6
- RN402 pad 4: /DE0-Nano/MOD0_D14 -> /DE0-Nano/MOD0_D7
- RN402 pad 5: Net-(J401-Pad15) -> /Module Headers/M0_D7
- RN402 pad 6: Net-(J401-Pad13) -> /Module Headers/M0_D6
- RN402 pad 7: Net-(J401-Pad11) -> /Module Headers/M0_D5
- RN402 pad 8: Net-(J401-Pad9) -> /Module Headers/M0_D4
- RN403 pad 1: Net-(J401-Pad2) -> /DE0-Nano/MOD0_D8
- RN403 pad 2: Net-(J401-Pad4) -> /DE0-Nano/MOD0_D9
- RN403 pad 3: Net-(J401-Pad6) -> /DE0-Nano/MOD0_D10
- RN403 pad 4: Net-(J401-Pad8) -> /DE0-Nano/MOD0_D11
- RN403 pad 5: /DE0-Nano/MOD0_D7 -> /Module Headers/M0_D11
- RN403 pad 6: /DE0-Nano/MOD0_D5 -> /Module Headers/M0_D10
- RN403 pad 7: /DE0-Nano/MOD0_D3 -> /Module Headers/M0_D9
- RN403 pad 8: /DE0-Nano/MOD0_D1 -> /Module Headers/M0_D8
- RN404 pad 1: Net-(J401-Pad10) -> /DE0-Nano/MOD0_D12
- RN404 pad 2: Net-(J401-Pad12) -> /DE0-Nano/MOD0_D13
- RN404 pad 3: Net-(J401-Pad14) -> /DE0-Nano/MOD0_D14
- RN404 pad 4: Net-(J401-Pad16) -> /DE0-Nano/MOD0_D15
- RN404 pad 5: /DE0-Nano/MOD0_D15 -> /Module Headers/M0_D15
- RN404 pad 6: /DE0-Nano/MOD0_D13 -> /Module Headers/M0_D14
- RN404 pad 7: /DE0-Nano/MOD0_D11 -> /Module Headers/M0_D13
- RN404 pad 8: /DE0-Nano/MOD0_D9 -> /Module Headers/M0_D12
- RN407 pad 1: Net-(J402-Pad2) -> /DE0-Nano/MOD1_D8
- RN407 pad 2: Net-(J402-Pad4) -> /DE0-Nano/MOD1_D9
- RN407 pad 3: Net-(J402-Pad6) -> /DE0-Nano/MOD1_D10
- RN407 pad 4: Net-(J402-Pad8) -> /DE0-Nano/MOD1_D11
- RN407 pad 5: /DE0-Nano/MOD1_D7 -> /Module Headers/M1_D11
- RN407 pad 6: /DE0-Nano/MOD1_D5 -> /Module Headers/M1_D10
- RN407 pad 7: /DE0-Nano/MOD1_D3 -> /Module Headers/M1_D9
- RN407 pad 8: /DE0-Nano/MOD1_D1 -> /Module Headers/M1_D8
- RN408 pad 1: Net-(J402-Pad10) -> /DE0-Nano/MOD1_D12
- RN408 pad 2: Net-(J402-Pad12) -> /DE0-Nano/MOD1_D13
- RN408 pad 3: Net-(J402-Pad14) -> /DE0-Nano/MOD1_D14
- RN408 pad 4: Net-(J402-Pad16) -> /DE0-Nano/MOD1_D15
- RN408 pad 5: /DE0-Nano/MOD1_D15 -> /Module Headers/M1_D15
- RN408 pad 6: /DE0-Nano/MOD1_D13 -> /Module Headers/M1_D14
- RN408 pad 7: /DE0-Nano/MOD1_D11 -> /Module Headers/M1_D13
- RN408 pad 8: /DE0-Nano/MOD1_D9 -> /Module Headers/M1_D12
Routing:
- net GND: track 0.00 -> 449.5 mm
- net +3.3VA: track 0.00 -> 122.4 mm, vias 0 -> 2
- net +5V: track 0.00 -> 110.2 mm
- net +5VA: track 0.00 -> 104.4 mm
- net /Cypress FX3/USB_CTL12: track 0.00 -> 61.5 mm
- net /Cypress FX3/USB_CTL11: track 0.00 -> 61.5 mm
- net /Cypress FX3/USB_CTL10: track 0.00 -> 55.5 mm
- net /Cypress FX3/USB_CTL9: track 0.00 -> 55.4 mm
- net /Cypress FX3/USB_CTL7: track 0.00 -> 49.3 mm
- net /Cypress FX3/USB_CTL8: track 0.00 -> 49.3 mm
- net /Cypress FX3/USB_CTL5: track 0.00 -> 43.5 mm
- net /Cypress FX3/USB_CTL6: track 0.00 -> 43.1 mm
- net /Cypress FX3/USB_CTL4: track 0.00 -> 37.1 mm
- net /Cypress FX3/USB_CTL3: track 0.00 -> 37.0 mm
- net /Cypress FX3/USB_DATA16: track 0.00 -> 31.6 mm
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Other:
- board outline added: 99.1 x 90.8 mm

Commit message: Finished base board ready for review
Parts:
- added G***: LOGO, Logo:DdD_logo, B.Cu at (182.2, 99.1)
- added G***: LOGO, Logo:oshw logo, B.Cu at (182.2, 118.7)
- added G***: LOGO, Logo:CC Licence, B.Cu at (115.6, 123.8)
- added G***: LOGO, Logo:dd86 logo, B.Cu at (184.8, 62.9)
- added G***: LOGO, Logo:CC Licence, F.Cu at (161.9, 95.2)
- added G***: LOGO, Logo:DdD_logo_square, F.Cu at (115.6, 58.4)
- added G***: LOGO, Logo:DdD_logo, F.Cu at (181.6, 94.6)
- moved FID602 5.08 mm to (202.2, 59.1)
- moved FID601 5.08 mm to (111.8, 53.0)
- moved FID603 5.00 mm to (111.3, 136.3)
Routing:
- net +5VA: track 104.4 -> 109.1 mm
- net /Cypress FX3/USB_CTL12: track 61.5 -> 63.7 mm
- net +3.3VA: track 122.4 -> 120.3 mm
- net /Cypress FX3/USB_CTL11: track 61.5 -> 63.6 mm
- net /Cypress FX3/USB_CTL9: track 55.4 -> 56.7 mm
- net /Cypress FX3/USB_CTL10: track 55.5 -> 56.8 mm
- net /Module Headers/M1_D3: track 20.7 -> 21.8 mm
- net /Module Headers/M0_D4: track 5.40 -> 6.45 mm
- net /Module Headers/M1_D4: track 16.1 -> 16.9 mm
- net /Module Headers/M1_D2: track 17.7 -> 18.4 mm
- net /Cypress FX3/USB_CTL8: track 49.3 -> 49.9 mm
- net /Module Headers/M1_D11: track 12.0 -> 12.7 mm
- net /Module Headers/M1_D7: track 20.4 -> 21.0 mm
- net /Cypress FX3/USB_CTL7: track 49.3 -> 49.9 mm
- net /Module Headers/M0_D5: track 8.41 -> 8.96 mm
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- added copper zone on B.Cu, net GND
- added copper zone on F.Cu, net GND
Other:
- board text added: "(C) 2019 Simon Inns - Attribution ShareAlike 4.0 International (CC BY-SA 4.0)"
- board text added: "Base Board Version 4_0"
- board text added: "Domesday Duplicator 4"
- board text added: "Key"
- board text added: "Module 0"
- board text added: "Module 1"
- board text added: "https://www.domesday86.com"
- board text added: "https://www.domesday86.com Recreating the Domesday Experience"

Commit message: Added ld-decode logo
Parts:
- removed the G*** at (182.2, 118.7)
- added G***: LOGO, Logo:ld-decode-logo, B.Cu at (114.3, 84.5)
- added REF**: OSHW-Logo2_14.6x12mm_SilkScreen, Symbol:OSHW-Logo2_14.6x12mm_SilkScreen, B.Cu at (182.9, 114.9)
- added REF**: OSHW-Logo2_14.6x12mm_SilkScreen, Symbol:OSHW-Logo2_14.6x12mm_SilkScreen, F.Cu at (186.7, 64.8)
- moved FID602 1.09 mm to (201.3, 59.7)
