File: Hardware/DomesdayDuplicator-module-ADS825/ADC.sch (KiCad schematic (older format))
At the start: 20 parts, among them U301 MCP602, U302 ADS825E

Commit message: Added DdD base DE0-Nano connections and part mapping for ADS825 module
Parts:
- C301, C303, C305, C307, C308, C311, C313, C315: footprint (none) -> Capacitor_SMD:C_0805_2012Metric
- C302, C304, C306, C309, C310, C312, C314, C316: footprint (none) -> Capacitor_Tantalum_SMD:CP_EIA-3216-18_Kemet-A
- R301, R302: footprint (none) -> Resistor_SMD:R_0805_2012Metric
- U301: footprint (none) -> Package_SO:SOIC-8_3.9x4.9mm_P1.27mm
- U302: footprint (none) -> Package_SO:SSOP-28_5.3x10.2mm_P0.65mm
Changed lines of the file:
@@
 F 0 "C316" H 7118 4496 50  0000 L CNN
 F 1 "2.2uF Tant" H 7118 4405 50  0000 L CNN
-F 2 "" H 7038 4300 50  0001 C CNN
+F 2 "Capacitor_Tantalum_SMD:CP_EIA-3216-18_Kemet-A" H 7038 4300 50  0001 C CNN
 F 3 "~" H 7000 4450 50  0001 C CNN
 	1    7000 4450
@@
 F 0 "C315" H 6665 4496 50  0000 L CNN
 F 1 "100nF" H 6665 4405 50  0000 L CNN
-F 2 "" H 6588 4300 50  0001 C CNN
+F 2 "Capacitor_SMD:C_0805_2012Metric" H 6588 4300 50  0001 C CNN
 F 3 "~" H 6550 4450 50  0001 C CNN
 	1    6550 4450
@@
 F 0 "C314" H 6518 4096 50  0000 L CNN
 F 1 "2.2uF Tant" H 6518 4005 50  0000 L CNN
-F 2 "" H 6438 3900 50  0001 C CNN
+F 2 "Capacitor_Tantalum_SMD:CP_EIA-3216-18_Kemet-A" H 6438 3900 50  0001 C CNN
 F 3 "~" H 6400 4050 50  0001 C CNN
 	1    6400 4050
@@
 F 0 "C313" H 6065 4096 50  0000 L CNN
 F 1 "100nF" H 6065 4005 50  0000 L CNN
-F 2 "" H 5988 3900 50  0001 C CNN
+F 2 "Capacitor_SMD:C_0805_2012Metric" H 5988 3900 50  0001 C CNN
 F 3 "~" H 5950 4050 50  0001 C CNN
 	1    5950 4050
@@
 F 0 "C312" H 5518 4496 50  0000 L CNN
 F 1 "2.2uF Tant" H 5518 4405 50  0000 L CNN
-F 2 "" H 5438 4300 50  0001 C CNN
+F 2 "Capacitor_Tantalum_SMD:CP_EIA-3216-18_Kemet-A" H 5438 4300 50  0001 C CNN
 F 3 "~" H 5400 4450 50  0001 C CNN
 	1    5400 4450
@@
 F 0 "C311" H 5065 4496 50  0000 L CNN
 F 1 "100nF" H 5065 4405 50  0000 L CNN
-F 2 "" H 4988 4300 50  0001 C CNN
+F 2 "Capacitor_SMD:C_0805_2012Metric" H 4988 4300 50  0001 C CNN
 F 3 "~" H 4950 4450 50  0001 C CNN
 	1    4950 4450
@@
 F 0 "C310" H 4918 4096 50  0000 L CNN
 F 1 "2.2uF Tant" H 4918 4005 50  0000 L CNN
-F 2 "" H 4838 3900 50  0001 C CNN
+F 2 "Capacitor_Tantalum_SMD:CP_EIA-3216-18_Kemet-A" H 4838 3900 50  0001 C CNN
 F 3 "~" H 4800 4050 50  0001 C CNN
 	1    4800 4050
@@
 F 0 "C308" H 4465 4096 50  0000 L CNN
 F 1 "100nF" H 4465 4005 50  0000 L CNN
-F 2 "" H 4388 3900 50  0001 C CNN
+F 2 "Capacitor_SMD:C_0805_2012Metric" H 4388 3900 50  0001 C CNN
 F 3 "~" H 4350 4050 50  0001 C CNN
 	1    4350 4050
@@
 F 0 "C306" H 3918 4496 50  0000 L CNN
 F 1 "2.2uF Tant" H 3918 4405 50  0000 L CNN
-F 2 "" H 3838 4300 50  0001 C CNN
+F 2 "Capacitor_Tantalum_SMD:CP_EIA-3216-18_Kemet-A" H 3838 4300 50  0001 C CNN
 F 3 "~" H 3800 4450 50  0001 C CNN
 	1    3800 4450
@@
 F 0 "C305" H 3465 4496 50  0000 L CNN
 F 1 "100nF" H 3465 4405 50  0000 L CNN
-F 2 "" H 3388 4300 50  0001 C CNN
+F 2 "Capacitor_SMD:C_0805_2012Metric" H 3388 4300 50  0001 C CNN
 F 3 "~" H 3350 4450 50  0001 C CNN
 	1    3350 4450
@@
 F 0 "R301" V 3193 3300 50  0000 C CNN
 F 1 "1K" V 3284 3300 50  0000 C CNN
-F 2 "" V 3330 3300 50  0001 C CNN
+F 2 "Resistor_SMD:R_0805_2012Metric" V 3330 3300 50  0001 C CNN
 F 3 "~" H 3400 3300 50  0001 C CNN
 	1    3400 3300
@@
 F 0 "R302" V 3193 3800 50  0000 C CNN
 F 1 "1K" V 3284 3800 50  0000 C CNN
-F 2 "" V 3330 3800 50  0001 C CNN
+F 2 "Resistor_SMD:R_0805_2012Metric" V 3330 3800 50  0001 C CNN
 F 3 "~" H 3400 3800 50  0001 C CNN
 	1    3400 3800
@@
 F 0 "C302" H 1868 6996 50  0000 L CNN
 F 1 "2.2uF Tant" H 1868 6905 50  0000 L CNN
-F 2 "" H 1788 6800 50  0001 C CNN
+F 2 "Capacitor_Tantalum_SMD:CP_EIA-3216-18_Kemet-A" H 1788 6800 50  0001 C CNN
 F 3 "~" H 1750 6950 50  0001 C CNN
 	1    1750 6950
@@
 F 0 "C301" H 1415 6996 50  0000 L CNN
 F 1 "100nF" H 1415 6905 50  0000 L CNN
-F 2 "" H 1338 6800 50  0001 C CNN
+F 2 "Capacitor_SMD:C_0805_2012Metric" H 1338 6800 50  0001 C CNN
 F 3 "~" H 1300 6950 50  0001 C CNN
 	1    1300 6950
@@
 F 0 "C304" H 2968 6996 50  0000 L CNN
 F 1 "2.2uF Tant" H 2968 6905 50  0000 L CNN
-F 2 "" H 2888 6800 50  0001 C CNN
+F 2 "Capacitor_Tantalum_SMD:CP_EIA-3216-18_Kemet-A" H 2888 6800 50  0001 C CNN
 F 3 "~" H 2850 6950 50  0001 C CNN
 	1    2850 6950
@@
 F 0 "C303" H 2515 6996 50  0000 L CNN
 F 1 "100nF" H 2515 6905 50  0000 L CNN
-F 2 "" H 2438 6800 50  0001 C CNN
+F 2 "Capacitor_SMD:C_0805_2012Metric" H 2438 6800 50  0001 C CNN
 F 3 "~" H 2400 6950 50  0001 C CNN
 	1    2400 6950
@@
 F 0 "C309" H 4818 6946 50  0000 L CNN
 F 1 "2.2uF Tant" H 4818 6855 50  0000 L CNN
-F 2 "" H 4738 6750 50  0001 C CNN
+F 2 "Capacitor_Tantalum_SMD:CP_EIA-3216-18_Kemet-A" H 4738 6750 50  0001 C CNN
 F 3 "~" H 4700 6900 50  0001 C CNN
 	1    4700 6900
@@
 F 0 "C307" H 4365 6946 50  0000 L CNN
 F 1 "100nF" H 4365 6855 50  0000 L CNN
-F 2 "" H 4288 6750 50  0001 C CNN
+F 2 "Capacitor_SMD:C_0805_2012Metric" H 4288 6750 50  0001 C CNN
 F 3 "~" H 4250 6900 50  0001 C CNN
 	1    4250 6900
@@
 F 0 "U301" H 2700 2433 50  0000 C CNN
 F 1 "MCP602" H 2700 2524 50  0000 C CNN
-F 2 "" H 2700 2800 50  0001 C CNN
+F 2 "Package_SO:SOIC-8_3.9x4.9mm_P1.27mm" H 2700 2800 50  0001 C CNN
 F 3 "http://ww1.microchip.com/downloads/en/DeviceDoc/21314g.pdf" H 2700 2800 50  0001 C CNN
 	1    2700 2800
@@
 F 0 "U301" H 2700 3333 50  0000 C CNN
 F 1 "MCP602" H 2700 3424 50  0000 C CNN
-F 2 "" H 2700 3700 50  0001 C CNN
+F 2 "Package_SO:SOIC-8_3.9x4.9mm_P1.27mm" H 2700 3700 50  0001 C CNN
 F 3 "http://ww1.microchip.com/downloads/en/DeviceDoc/21314g.pdf" H 2700 3700 50  0001 C CNN
 	2    2700 3700
@@
 F 0 "U301" H 808 6996 50  0000 L CNN
 F 1 "MCP602" H 808 6905 50  0000 L CNN
-F 2 "" H 850 6950 50  0001 C CNN
+F 2 "Package_SO:SOIC-8_3.9x4.9mm_P1.27mm" H 850 6950 50  0001 C CNN
 F 3 "http://ww1.microchip.com/downloads/en/DeviceDoc/21314g.pdf" H 850 6950 50  0001 C CNN
 	3    850  6950
@@
 Text Label 8900 3850 0    50   ~ 0
 DO9
-Wire Bus Line
-	9350 2800 9350 3950
 $Comp
 L Domesday-Duplicator-module-library:ADS825E U302
@@
 F 0 "U302" H 7900 4400 50  0000 C CNN
 F 1 "ADS825E" H 8650 4400 50  0000 C CNN
-F 2 "" H 9050 3250 50  0001 C CNN
+F 2 "Package_SO:SSOP-28_5.3x10.2mm_P0.65mm" H 9050 3250 50  0001 C CNN
 F 3 "" H 9050 3250 50  0001 C CNN
 	1    8300 3600
 	1    0    0    -1
 $EndComp
+Wire Bus Line
+	9350 2800 9350 3950
 $EndSCHEMATC
