File: Hardware/DomesdayDuplicator-module-ADS825/DomesdayDuplicator-module-ADS825.sch (KiCad schematic (older format))
At the start: 0 parts

Commit message: Fixes to module and base - added component mapping to base and verified mirrored headers
Changed lines of the file:
@@
 $Descr A4 11693 8268
 encoding utf-8
-Sheet 1 6
+Sheet 1 7
 Title "Domesday Duplicator Module - ADS825"
 Date "2019-09-02"
@@
 $EndDescr
 $Sheet
-S 3100 3650 1000 300
+S 3100 3400 1000 300
 U 5D6B6623
 F0 "RF Front-End" 50
 F1 "rf-front-end.sch" 50
-F2 "RF_OUT" O R 4100 3750 50
-F3 "DC_OFFSET" I R 4100 3850 50
+F2 "RF_OUT" O R 4100 3500 50
+F3 "DC_OFFSET" I R 4100 3600 50
 $EndSheet
 $Sheet
-S 4700 3650 1000 300
+S 4700 3400 1000 300
 U 5D7040C0
 F0 "ADC" 50
 F1 "ADC.sch" 50
-F2 "DO[0..9]" O R 5700 3750 50
-F3 "CLK" I R 5700 3850 50
-F4 "DC_OFFSET" O L 4700 3850 50
-F5 "ANALOG_IN" I L 4700 3750 50
+F2 "DO[0..9]" O R 5700 3500 50
+F3 "CLK" I R 5700 3600 50
+F4 "DC_OFFSET" O L 4700 3600 50
+F5 "ANALOG_IN" I L 4700 3500 50
 $EndSheet
 Wire Wire Line
-	4100 3750 4700 3750
+	4100 3500 4700 3500
 Wire Wire Line
-	4700 3850 4100 3850
+	4700 3600 4100 3600
 $Sheet
-S 6200 3650 1000 300
+S 6200 3400 1000 300
 U 5D7B659B
 F0 "Line Drivers" 50
 F1 "line-drivers.sch" 50
-F2 "TRIGGER_IN" I L 6200 3850 50
-F3 "DO[0..9]" I L 6200 3750 50
-F4 "DB[0..10]" O R 7200 3750 50
+F2 "TRIGGER_IN" I L 6200 3600 50
+F3 "DO[0..9]" I L 6200 3500 50
+F4 "DB[0..10]" O R 7200 3500 50
 $EndSheet
 Wire Bus Line
-	5700 3750 6200 3750
+	5700 3500 6200 3500
 $Sheet
-S 3100 4200 1000 300
+S 3100 3950 1000 300
 U 5D80DE2B
 F0 "Trigger Input" 50
 F1 "trigger-input.sch" 50
-F2 "TRIGGER_OUT" O R 4100 4300 50
+F2 "TRIGGER_OUT" O R 4100 4050 50
 $EndSheet
 Wire Wire Line
-	4100 4300 6100 4300
+	4100 4050 6100 4050
 Wire Wire Line
-	6100 4300 6100 3850
+	6100 4050 6100 3600
 Wire Wire Line
-	6100 3850 6200 3850
+	6100 3600 6200 3600
 $Sheet
-S 7900 3650 1000 300
+S 7900 3400 1000 300
 U 5D81734A
 F0 "Header" 50
 F1 "header.sch" 50
-F2 "CLK" O L 7900 3850 50
-F3 "DB[0..10]" I L 7900 3750 50
+F2 "CLK" O L 7900 3600 50
+F3 "DB[0..10]" I L 7900 3500 50
 $EndSheet
 Wire Bus Line
-	7200 3750 7900 3750
+	7200 3500 7900 3500
 Wire Wire Line
-	5700 3850 5800 3850
+	5700 3600 5800 3600
 Wire Wire Line
-	5800 3850 5800 4200
+	5800 3600 5800 3950
 Wire Wire Line
-	5800 4200 7800 4200
+	5800 3950 7800 3950
 Wire Wire Line
-	7800 4200 7800 3850
+	7800 3950 7800 3600
 Wire Wire Line
-	7800 3850 7900 3850
+	7800 3600 7900 3600
+$Sheet
+S 4700 6450 900  1050
+U 5D70405C
+F0 "Fiducials and Mounting" 50
+F1 "fiducials-mounting.sch" 50
+$EndSheet
 $EndSCHEMATC
