File: Hardware/DomesdayDuplicator-module-ADS825/line-drivers.sch (KiCad schematic (older format))
At the start: 6 parts, among them U401 74LVTH541, U402 74LVTH541

Commit message: Added DdD base DE0-Nano connections and part mapping for ADS825 module
Parts:
- removed C402, C404: 2.2uF Tant, symbol Device:CP
- C401: footprint (none) -> Capacitor_SMD:C_0805_2012Metric
- C402: renamed from C403; footprint (none) -> Capacitor_SMD:C_0805_2012Metric
- U401, U402: footprint (none) -> Package_SO:SSOP-20_4.4x6.5mm_P0.65mm
Other:
- moved on the sheet: C402
Changed lines of the file:
@@
 F 0 "U401" H 6150 2000 50  0000 C CNN
 F 1 "74LVTH541" H 6150 3300 50  0000 C CNN
-F 2 "" H 5900 2650 50  0001 C CNN
+F 2 "Package_SO:SSOP-20_4.4x6.5mm_P0.65mm" H 5900 2650 50  0001 C CNN
 F 3 "http://www.ti.com/lit/gpn/sn74HCT541" H 5900 2650 50  0001 C CNN
 	1    5900 2650
@@
 F 0 "U402" H 6150 4250 50  0000 C CNN
 F 1 "74LVTH541" H 6150 5550 50  0000 C CNN
-F 2 "" H 5900 4900 50  0001 C CNN
+F 2 "Package_SO:SSOP-20_4.4x6.5mm_P0.65mm" H 5900 4900 50  0001 C CNN
 F 3 "http://www.ti.com/lit/gpn/sn74HCT541" H 5900 4900 50  0001 C CNN
 	1    5900 4900
@@
 NoConn ~ 6400 5100
 $Comp
-L Device:CP C?
-U 1 1 5D7DBDC7
-P 1250 7100
-AR Path="/5D7040C0/5D7DBDC7" Ref="C?"  Part="1"
-AR Path="/5D7B659B/5D7DBDC7" Ref="C402"  Part="1"
-F 0 "C402" H 1368 7146 50  0000 L CNN
-F 1 "2.2uF Tant" H 1368 7055 50  0000 L CNN
-F 2 "" H 1288 6950 50  0001 C CNN
-F 3 "~" H 1250 7100 50  0001 C CNN
-	1    1250 7100
-	1    0    0    -1
-$EndComp
-$Comp
 L Device:C C?
 U 1 1 5D7DBDCD
@@
 F 0 "C401" H 915 7146 50  0000 L CNN
 F 1 "100nF" H 915 7055 50  0000 L CNN
-F 2 "" H 838 6950 50  0001 C CNN
+F 2 "Capacitor_SMD:C_0805_2012Metric" H 838 6950 50  0001 C CNN
 F 3 "~" H 800 7100 50  0001 C CNN
 	1    800  7100
@@
 Wire Wire Line
 	800  6950 800  6850
-Wire Wire Line
-	800  6850 1250 6850
-Wire Wire Line
-	1250 6850 1250 6950
 Connection ~ 800  6850
 Wire Wire Line
 	800  6850 800  6800
-Wire Wire Line
-	1250 7250 1250 7350
-Wire Wire Line
-	1250 7350 800  7350
 Connection ~ 800  7350
 Wire Wire Line
 	800  7350 800  7250
-$Comp
-L Device:CP C?
-U 1 1 5D7DD74B
-P 2350 7100
-AR Path="/5D7040C0/5D7DD74B" Ref="C?"  Part="1"
-AR Path="/5D7B659B/5D7DD74B" Ref="C404"  Part="1"
-F 0 "C404" H 2468 7146 50  0000 L CNN
-F 1 "2.2uF Tant" H 2468 7055 50  0000 L CNN
-F 2 "" H 2388 6950 50  0001 C CNN
-F 3 "~" H 2350 7100 50  0001 C CNN
-	1    2350 7100
-	1    0    0    -1
-$EndComp
 $Comp
 L Device:C C?
 U 1 1 5D7DD755
-P 1900 7100
+P 1300 7100
 AR Path="/5D7040C0/5D7DD755" Ref="C?"  Part="1"
-AR Path="/5D7B659B/5D7DD755" Ref="C403"  Part="1"
-F 0 "C403" H 2015 7146 50  0000 L CNN
-F 1 "100nF" H 2015 7055 50  0000 L CNN
-F 2 "" H 1938 6950 50  0001 C CNN
-F 3 "~" H 1900 7100 50  0001 C CNN
-	1    1900 7100
-	1    0    0    -1
-$EndComp
-Wire Wire Line
-	1900 6950 1900 6850
-Wire Wire Line
-	2350 6850 2350 6950
-Wire Wire Line
-	2350 7250 2350 7350
-Wire Wire Line
-	1900 7350 1900 7250
-Wire Wire Line
-	1250 7350 1900 7350
-Connection ~ 1250 7350
-Wire Wire Line
-	1900 7350 2350 7350
-Connection ~ 1900 7350
-Wire Wire Line
-	2350 6850 1900 6850
-Wire Wire Line
-	1900 6850 1250 6850
-Connection ~ 1900 6850
-Connection ~ 1250 6850
+AR Path="/5D7B659B/5D7DD755" Ref="C402"  Part="1"
+F 0 "C402" H 1415 7146 50  0000 L CNN
+F 1 "100nF" H 1415 7055 50  0000 L CNN
+F 2 "Capacitor_SMD:C_0805_2012Metric" H 1338 6950 50  0001 C CNN
+F 3 "~" H 1300 7100 50  0001 C CNN
+	1    1300 7100
+	1    0    0    -1
+$EndComp
+Wire Wire Line
+	1300 6950 1300 6850
+Wire Wire Line
+	1300 7350 1300 7250
 Text Label 5200 2150 0    50   ~ 0
 DO0
@@
 TRIGGER_IN
 NoConn ~ 6400 4700
+Wire Wire Line
+	800  6850 1300 6850
+Wire Wire Line
+	800  7350 1300 7350
 Wire Bus Line
 	5050 2050 5050 4400
