File: Hardware/DomesdayDuplicator-module-ADS825/header.sch (KiCad schematic (older format))
At the start: 2 parts, among them J601 Conn_02x10_Odd_Even, J602 Conn_02x10_Odd_Even

Commit message: Added DdD base DE0-Nano connections and part mapping for ADS825 module
Parts:
- J601: value Conn_02x10_Odd_Even -> Back_connector; footprint (none) -> Connector_PinHeader_1.27mm:PinHeader_2x10_P1.27mm_Vertical_SMD
- J602: value Conn_02x10_Odd_Even -> Front_connector; footprint (none) -> Connector_PinHeader_1.27mm:PinHeader_2x10_P1.27mm_Vertical_SMD
Connections:
- net +3V3: now also J601.2 (Pin_2); no longer J601.19 (Pin_19)
- net +5VA: now also J601.3 (Pin_3); no longer J601.18 (Pin_18)
- net CLK: now also J601.4 (Pin_4); no longer J601.17 (Pin_17)
- net DB0: now also J601.20 (Pin_20); no longer J601.1 (Pin_1)
- net DB1: now also J601.19 (Pin_19); no longer J601.2 (Pin_2)
- net DB10: now also J601.10 (Pin_10); no longer J601.11 (Pin_11)
- net DB2: now also J601.18 (Pin_18); no longer J601.3 (Pin_3)
- net DB3: now also J601.17 (Pin_17); no longer J601.4 (Pin_4)
- net DB4: now also J601.16 (Pin_16); no longer J601.5 (Pin_5)
- net DB5: now also J601.15 (Pin_15); no longer J601.6 (Pin_6)
- net DB6: now also J601.14 (Pin_14); no longer J601.7 (Pin_7)
- net DB7: now also J601.13 (Pin_13); no longer J601.8 (Pin_8)
- net DB8: now also J601.12 (Pin_12); no longer J601.9 (Pin_9)
- net DB9: now also J601.11 (Pin_11); no longer J601.10 (Pin_10)
- net GND: now also J601.1 (Pin_1); no longer J601.20 (Pin_20)
Other:
- moved on the sheet: J602
Changed lines of the file:
@@
 L Connector_Generic:Conn_02x10_Odd_Even J601
 U 1 1 5D6D02A7
-P 5200 4000
-F 0 "J601" H 5250 4617 50  0000 C CNN
-F 1 "Conn_02x10_Odd_Even" H 5250 4526 50  0000 C CNN
-F 2 "" H 5200 4000 50  0001 C CNN
-F 3 "~" H 5200 4000 50  0001 C CNN
-	1    5200 4000
-	1    0    0    -1
+P 5300 4100
+F 0 "J601" H 5350 4717 50  0000 C CNN
+F 1 "Back_connector" H 5350 4626 50  0000 C CNN
+F 2 "Connector_PinHeader_1.27mm:PinHeader_2x10_P1.27mm_Vertical_SMD" H 5300 4100 50  0001 C CNN
+F 3 "~" H 5300 4100 50  0001 C CNN
+	1    5300 4100
+	-1   0    0    1
 $EndComp
 $Comp
 L Connector_Generic:Conn_02x10_Odd_Even J602
 U 1 1 5D6D0FBD
-P 7650 4000
-F 0 "J602" H 7700 4617 50  0000 C CNN
-F 1 "Conn_02x10_Odd_Even" H 7700 4526 50  0000 C CNN
-F 2 "" H 7650 4000 50  0001 C CNN
-F 3 "~" H 7650 4000 50  0001 C CNN
-	1    7650 4000
-	1    0    0    -1
+P 8000 4050
+F 0 "J602" H 8050 4667 50  0000 C CNN
+F 1 "Front_connector" H 8050 4576 50  0000 C CNN
+F 2 "Connector_PinHeader_1.27mm:PinHeader_2x10_P1.27mm_Vertical_SMD" H 8000 4050 50  0001 C CNN
+F 3 "~" H 8000 4050 50  0001 C CNN
+	1    8000 4050
+	-1   0    0    1
 $EndComp
 Wire Wire Line
@@
 Text Label 5500 4500 0    50   ~ 0
 GND
-NoConn ~ 7450 3600
-NoConn ~ 7450 3700
-NoConn ~ 7450 3800
-NoConn ~ 7450 3900
-NoConn ~ 7450 4000
-NoConn ~ 7450 4100
-NoConn ~ 7450 4200
-NoConn ~ 7450 4300
-NoConn ~ 7450 4400
-NoConn ~ 7450 4500
-NoConn ~ 7950 3600
-NoConn ~ 7950 3700
-NoConn ~ 7950 3800
-NoConn ~ 7950 3900
-NoConn ~ 7950 4000
-NoConn ~ 7950 4100
-NoConn ~ 7950 4200
-NoConn ~ 7950 4300
-NoConn ~ 7950 4400
-NoConn ~ 7950 4500
+NoConn ~ 8200 4450
+NoConn ~ 8200 4350
+NoConn ~ 8200 4250
+NoConn ~ 8200 4150
+NoConn ~ 8200 4050
+NoConn ~ 8200 3950
+NoConn ~ 8200 3850
+NoConn ~ 8200 3750
+NoConn ~ 8200 3650
+NoConn ~ 8200 3550
+NoConn ~ 7700 4450
+NoConn ~ 7700 4350
+NoConn ~ 7700 4250
+NoConn ~ 7700 4150
+NoConn ~ 7700 4050
+NoConn ~ 7700 3950
+NoConn ~ 7700 3850
+NoConn ~ 7700 3750
+NoConn ~ 7700 3650
+NoConn ~ 7700 3550
 NoConn ~ 5500 4100
 NoConn ~ 5500 4200
@@
 	4250 4500 5000 4500
 $Comp
-L power:PWR_FLAG #FLG0101
+L power:PWR_FLAG #FLG0602
 U 1 1 5D704F07
 P 6500 4200
-F 0 "#FLG0101" H 6500 4275 50  0001 C CNN
+F 0 "#FLG0602" H 6500 4275 50  0001 C CNN
 F 1 "PWR_FLAG" H 6500 4373 50  0000 C CNN
 F 2 "" H 6500 4200 50  0001 C CNN
@@
 $EndComp
 $Comp
-L power:PWR_FLAG #FLG0102
+L power:PWR_FLAG #FLG0601
 U 1 1 5D705FDB
 P 3900 4200
-F 0 "#FLG0102" H 3900 4275 50  0001 C CNN
+F 0 "#FLG0601" H 3900 4275 50  0001 C CNN
 F 1 "PWR_FLAG" H 3900 4373 50  0000 C CNN
 F 2 "" H 3900 4200 50  0001 C CNN
@@
 Connection ~ 6100 4500
 $Comp
-L power:GND #PWR0101
+L power:GND #PWR0604
 U 1 1 5D70D0A7
 P 6500 4650
-F 0 "#PWR0101" H 6500 4400 50  0001 C CNN
+F 0 "#PWR0604" H 6500 4400 50  0001 C CNN
 F 1 "GND" H 6505 4477 50  0000 C CNN
 F 2 "" H 6500 4650 50  0001 C CNN
@@
 $EndComp
 $Comp
-L power:PWR_FLAG #FLG0103
+L power:PWR_FLAG #FLG0603
 U 1 1 5D70D260
 P 6900 4650
-F 0 "#FLG0103" H 6900 4725 50  0001 C CNN
+F 0 "#FLG0603" H 6900 4725 50  0001 C CNN
 F 1 "PWR_FLAG" H 6900 4823 50  0000 C CNN
 F 2 "" H 6900 4650 50  0001 C CNN

Commit message: Work on the ADS825 module to determine the overall module dimensions and mounting
Parts:
- removed J602: Front_connector, Connector_PinHeader_1.27mm:PinHeader_2x10_P1.27mm_Vertical_SMD, symbol Connector_Generic:Conn_02x10_Odd_Even
- J601: value Back_connector -> Module_Connector; footprint Connector_PinHeader_1.27mm:PinHeader_2x10_P1.27mm_Vertical_SMD -> Connector_PinSocket_2.54mm:PinSocket_2x10_P2.54mm_Vertical
Connections:
- net +3V3: now also J601.19 (Pin_19); no longer J601.2 (Pin_2)
- net +5VA: now also J601.18 (Pin_18); no longer J601.3 (Pin_3)
- net CLK: now also J601.17 (Pin_17); no longer J601.4 (Pin_4)
- net DB0: now also J601.1 (Pin_1); no longer J601.20 (Pin_20)
- net DB1: now also J601.2 (Pin_2); no longer J601.19 (Pin_19)
- net DB10: now also J601.11 (Pin_11); no longer J601.10 (Pin_10)
- net DB2: now also J601.3 (Pin_3); no longer J601.18 (Pin_18)
- net DB3: now also J601.4 (Pin_4); no longer J601.17 (Pin_17)
- net DB4: now also J601.5 (Pin_5); no longer J601.16 (Pin_16)
- net DB5: now also J601.6 (Pin_6); no longer J601.15 (Pin_15)
- net DB6: now also J601.7 (Pin_7); no longer J601.14 (Pin_14)
- net DB7: now also J601.8 (Pin_8); no longer J601.13 (Pin_13)
- net DB8: now also J601.9 (Pin_9); no longer J601.12 (Pin_12)
- net DB9: now also J601.10 (Pin_10); no longer J601.11 (Pin_11)
- net GND: now also J601.20 (Pin_20); no longer J601.1 (Pin_1)
- no-connect marks 25 -> 5
Other:
- moved on the sheet: J601
