File: Hardware/DomesdayDuplicator-module-ADS825/DomesdayDuplicator-module-ADS825.kicad_pcb (KiCad board)
At the start: 2 copper layers, 57 parts, among them J201 RF_In_50R, J501 Trigger_In_50R, J601 Back_connector, J602 Front_connector, SW201 Gain_Select, U201 OPA690IDBVT, U301 MCP602, U302 ADS825E, U401 74LVTH541, U402 74LVTH541, U501 TLV3501

Commit message: Fixes to module and base - added component mapping to base and verified mirrored headers
Parts:
- added FID701: Fiducial, Fiducial:Fiducial_0.5mm_Dia_1mm_Outer, F.Cu at (159.5, 82.3)
- added FID702: Fiducial, Fiducial:Fiducial_0.5mm_Dia_1mm_Outer, F.Cu at (167.1, 82.3)
- added FID703: Fiducial, Fiducial:Fiducial_0.5mm_Dia_1mm_Outer, F.Cu at (174.5, 82.3)
Changed lines of the file:
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@@
     (tracks 0)
     (zones 0)
-    (modules 57)
+    (modules 60)
     (nets 52)
   )
@@
     )
   )
+  (module Fiducial:Fiducial_0.5mm_Dia_1mm_Outer (layer F.Cu)
+    (at 159.525001 82.309001)
+    (descr "Circular Fiducial, 0.5mm bare copper top, 1mm keepout (Level C)")
+    (tags fiducial)
+    (attr smd)
+    (fp_text reference FID701 (at 0 -1.5) (layer F.SilkS)
+      (effects (font (size 1 1) (thickness 0.15)))
+    )
+    (fp_text value Fiducial (at 0 1.5) (layer F.Fab)
+      (effects (font (size 1 1) (thickness 0.15)))
+    )
+    (fp_circle (center 0 0) (end 0.5 0) (layer F.Fab) (width 0.1))
+    (fp_text user %R (at 0 0) (layer F.Fab)
+      (effects (font (size 0.2 0.2) (thickness 0.04)))
+    )
+    (fp_circle (center 0 0) (end 0.75 0) (layer F.CrtYd) (width 0.05))
+    (pad "" smd circle (at 0 0) (size 0.5 0.5) (layers F.Cu F.Mask)
+      (solder_mask_margin 0.25) (clearance 0.25))
+  )
+  (module Fiducial:Fiducial_0.5mm_Dia_1mm_Outer (layer F.Cu)
+    (at 167.132 82.296)
+    (descr "Circular Fiducial, 0.5mm bare copper top, 1mm keepout (Level C)")
+    (tags fiducial)
+    (attr smd)
+    (fp_text reference FID702 (at 0 -1.5) (layer F.SilkS)
+      (effects (font (size 1 1) (thickness 0.15)))
+    )
+    (fp_text value Fiducial (at 0 1.5) (layer F.Fab)
+      (effects (font (size 1 1) (thickness 0.15)))
+    )
+    (fp_circle (center 0 0) (end 0.5 0) (layer F.Fab) (width 0.1))
+    (fp_text user %R (at 0 0) (layer F.Fab)
+      (effects (font (size 0.2 0.2) (thickness 0.04)))
+    )
+    (fp_circle (center 0 0) (end 0.75 0) (layer F.CrtYd) (width 0.05))
+    (pad "" smd circle (at 0 0) (size 0.5 0.5) (layers F.Cu F.Mask)
+      (solder_mask_margin 0.25) (clearance 0.25))
+  )
+  (module Fiducial:Fiducial_0.5mm_Dia_1mm_Outer (layer F.Cu)
+    (at 174.498 82.296)
+    (descr "Circular Fiducial, 0.5mm bare copper top, 1mm keepout (Level C)")
+    (tags fiducial)
+    (attr smd)
+    (fp_text reference FID703 (at 0 -1.5) (layer F.SilkS)
+      (effects (font (size 1 1) (thickness 0.15)))
+    )
+    (fp_text value Fiducial (at 0 1.5) (layer F.Fab)
+      (effects (font (size 1 1) (thickness 0.15)))
+    )
+    (fp_circle (center 0 0) (end 0.75 0) (layer F.CrtYd) (width 0.05))
+    (fp_text user %R (at 0 0) (layer F.Fab)
+      (effects (font (size 0.2 0.2) (thickness 0.04)))
+    )
+    (fp_circle (center 0 0) (end 0.5 0) (layer F.Fab) (width 0.1))
+    (pad "" smd circle (at 0 0) (size 0.5 0.5) (layers F.Cu F.Mask)
+      (solder_mask_margin 0.25) (clearance 0.25))
+  )
 )

Commit message: Work on the ADS825 module to determine the overall module dimensions and mounting
Parts:
- removed J602: Front_connector, Connector_PinHeader_1.27mm:PinHeader_2x10_P1.27mm_Vertical_SMD
- added H701: MountingHole, MountingHole:MountingHole_2.2mm_M2, F.Cu at (132.1, 90.9)
- J601: value Back_connector -> Module_Connector; footprint Connector_PinHeader_1.27mm:PinHeader_2x10_P1.27mm_Vertical_SMD -> Connector_PinSocket_2.54mm:PinSocket_2x10_P2.54mm_Vertical
- SW201: footprint Package_DIP:SMDIP-8_W7.62mm -> Button_Switch_SMD:SW_DIP_SPSTx04_Slide_Copal_CHS-04B_W7.62mm_P1.27mm
- moved R301 72.5 mm to (141.0, 102.4), turned to 90 degrees
- moved J601 71.1 mm to (164.5, 79.5), turned to 180 degrees
- moved C301 68.8 mm to (132.7, 106.4), turned to 90 degrees
- moved C309 67.6 mm to (152.5, 87.9)
- moved C401 67.6 mm to (157.9, 75.4)
- moved U302 67.6 mm to (149.2, 80.0)
- moved C303 67.6 mm to (148.2, 87.4)
- moved C304 67.6 mm to (145.9, 87.9)
- moved C307 67.6 mm to (150.2, 87.4)
- moved C402 67.6 mm to (158.1, 84.6)
- moved U401 67.6 mm to (158.1, 80.0)
- moved U402 67.6 mm to (158.1, 89.2)
- moved C302 66.9 mm to (132.7, 102.4), turned to 270 degrees
- moved R302 66.8 mm to (141.0, 106.2), turned to 90 degrees
- moved C306 66.8 mm to (138.2, 82.0), turned to 270 degrees
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Connections:
- J601 pad 1: GND -> /Header/DB0
- J601 pad 10: /Header/DB10 -> /Header/DB9
- J601 pad 11: /Header/DB9 -> /Header/DB10
- J601 pad 12: /Header/DB8 -> (no net)
- J601 pad 13: /Header/DB7 -> (no net)
- J601 pad 14: /Header/DB6 -> (no net)
- J601 pad 15: /Header/DB5 -> (no net)
- J601 pad 16: /Header/DB4 -> (no net)
- J601 pad 17: /Header/DB3 -> /ADC/CLK
- J601 pad 18: /Header/DB2 -> +5VA
- J601 pad 19: /Header/DB1 -> +3V3
- J601 pad 2: +3V3 -> /Header/DB1
- J601 pad 20: /Header/DB0 -> GND
- J601 pad 3: +5VA -> /Header/DB2
- J601 pad 4: /ADC/CLK -> /Header/DB3
- J601 pad 5: (no net) -> /Header/DB4
- J601 pad 6: (no net) -> /Header/DB5
- J601 pad 7: (no net) -> /Header/DB6
- J601 pad 8: (no net) -> /Header/DB7
- J601 pad 9: (no net) -> /Header/DB8
Other:
- board outline added: 49.5 x 38.1 mm

Commit message: Added ADC module complete with routing
Parts:
- added G***: LOGO, Logo:dd86 logo, B.Cu at (151.6, 83.3)
- added G***: LOGO, Logo:DdD_logo_square, F.Cu at (155.7, 99.3)
- added REF**: OSHW-Logo2_9.8x8mm_SilkScreen, Symbol:OSHW-Logo2_9.8x8mm_SilkScreen, B.Cu at (134.9, 96.8)
- J201, J501: footprint Connector_Coaxial:SMA_Amphenol_132289_EdgeMount -> digikey-footprints:RF_SMA_RightAngle_5-1814400-1
- moved R501 35.1 mm to (129.8, 81.0), turned to 270 degrees
- moved FID701 32.9 mm to (123.4, 108.0)
- moved C502 32.4 mm to (131.1, 75.7), turned to 180 degrees
- moved C501 31.8 mm to (131.6, 78.0), turned to 180 degrees
- moved R502 31.3 mm to (134.6, 84.3)
- moved U501 30.7 mm to (132.8, 81.0), turned to 0 degrees
- moved R503 28.3 mm to (130.8, 84.3), turned to 0 degrees
- moved R201 26.1 mm to (123.7, 105.2), turned to 180 degrees
- moved RV501 23.1 mm to (140.2, 86.9), turned to 270 degrees
- moved C201 21.9 mm to (127.3, 105.2), turned to 180 degrees
- moved C204 21.7 mm to (131.3, 103.6), turned to 180 degrees
- moved R203 20.3 mm to (127.3, 107.4), turned to 180 degrees
- moved U201 20.3 mm to (131.1, 106.7), turned to 0 degrees
- moved R302 20.3 mm to (134.6, 86.9), turned to 180 degrees
- moved R208 19.5 mm to (134.4, 101.6), turned to 180 degrees
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Routing:
- net GND: track 0.00 -> 349.4 mm, vias 0 -> 35
- net +5VA: track 0.00 -> 155.3 mm, vias 0 -> 9
- net +3V3: track 0.00 -> 73.1 mm, vias 0 -> 3
- net Net-(C308-Pad1): track 0.00 -> 37.2 mm, vias 0 -> 3
- net /ADC/CLK: track 0.00 -> 36.6 mm, vias 0 -> 1
- net /Line Drivers/TRIGGER_IN: track 0.00 -> 36.5 mm, vias 0 -> 2
- net Net-(U301-Pad6): track 0.00 -> 29.0 mm
- net /ADC/ANALOG_IN: track 0.00 -> 24.2 mm
- net Net-(C305-Pad1): track 0.00 -> 23.1 mm, vias 0 -> 3
- net Net-(R202-Pad2): track 0.00 -> 22.2 mm
- net /ADC/DC_OFFSET: track 0.00 -> 19.9 mm
- net Net-(R208-Pad2): track 0.00 -> 16.1 mm
- net Net-(C208-Pad1): track 0.00 -> 14.9 mm
- net Net-(R301-Pad2): track 0.00 -> 13.4 mm
- net Net-(C313-Pad1): track 0.00 -> 12.9 mm, vias 0 -> 2
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- added copper zone on B.Cu, net GND
- added copper zone on F.Cu, net GND
Other:
- board text added: "(C) 2019 Simon Inns"
- board text added: "40 MSPS ADC Module with Trigger"
- board text added: "Attribution-ShareAlike 4.0 International (CC BY-SA)"
- board text added: "Domesday Duplicator 4"
- board text added: "RF"
- board text added: "Trig"
- board text added: "V4_0"
- board text added: "https://www.domesday86.com"
- board text added: "https://www.domesday86.com Recreating the Domesday Experience"
- board text added: "o"
