File: Hardware/DomesdayDuplicator-module-ADS825/rf-front-end.sch (KiCad schematic (older format))
At the start: 23 parts, among them J201 RF_In_50R, SW201 Gain_Select, U201 OPA690IDBVT

Commit message: Added DdD base DE0-Nano connections and part mapping for ADS825 module
Parts:
- C201, C202, C203, C205, C206, C207, C208, C209: footprint (none) -> Capacitor_SMD:C_0805_2012Metric
- C204: footprint (none) -> Capacitor_Tantalum_SMD:CP_EIA-3216-18_Kemet-A
- J201: footprint (none) -> Connector_Coaxial:SMA_Amphenol_132289_EdgeMount
- L201, L202: footprint (none) -> Inductor_SMD:L_0805_2012Metric
- R201, R202, R203, R204, R205, R206, R207, R208, R209: footprint (none) -> Resistor_SMD:R_0805_2012Metric
- SW201: footprint (none) -> Package_DIP:SMDIP-8_W7.62mm
Other:
- note added: "2N Elliptic Filter (14 MHz low-pass)"
- note added: "Filter capactors should be 5% tolerance"
- note added: "Note:\nThe cable terminating resistor should\ntake into account the parallel resistance of\nthe dividing network:\n\n1000 / 2 = 500 Ohms\n\nRtotal = R1 x R2 / (R1 + R2)\n(500 * 56) / (500 + 56) = 50.36 Ohms"
Changed lines of the file:
@@
 F 0 "J201" H 2828 3388 50  0000 C CNN
 F 1 "RF_In_50R" H 2828 3297 50  0000 C CNN
-F 2 "" H 2900 3150 50  0001 C CNN
+F 2 "Connector_Coaxial:SMA_Amphenol_132289_EdgeMount" H 2900 3150 50  0001 C CNN
 F 3 " ~" H 2900 3150 50  0001 C CNN
 	1    2900 3150
@@
 F 0 "R201" H 3470 3396 50  0000 L CNN
 F 1 "56R" H 3470 3305 50  0000 L CNN
-F 2 "" V 3330 3350 50  0001 C CNN
+F 2 "Resistor_SMD:R_0805_2012Metric" V 3330 3350 50  0001 C CNN
 F 3 "~" H 3400 3350 50  0001 C CNN
 	1    3400 3350
@@
 F 0 "C201" V 3498 3150 50  0000 C CNN
 F 1 "100nF" V 3589 3150 50  0000 C CNN
-F 2 "" H 3788 3000 50  0001 C CNN
+F 2 "Capacitor_SMD:C_0805_2012Metric" H 3788 3000 50  0001 C CNN
 F 3 "~" H 3750 3150 50  0001 C CNN
 	1    3750 3150
@@
 F 0 "R203" V 4343 3150 50  0000 C CNN
 F 1 "100R" V 4434 3150 50  0000 C CNN
-F 2 "" V 4480 3150 50  0001 C CNN
+F 2 "Resistor_SMD:R_0805_2012Metric" V 4480 3150 50  0001 C CNN
 F 3 "~" H 4550 3150 50  0001 C CNN
 	1    4550 3150
@@
 F 0 "C202" V 4148 4900 50  0000 C CNN
 F 1 "100nF" V 4239 4900 50  0000 C CNN
-F 2 "" H 4438 4750 50  0001 C CNN
+F 2 "Capacitor_SMD:C_0805_2012Metric" H 4438 4750 50  0001 C CNN
 F 3 "~" H 4400 4900 50  0001 C CNN
 	1    4400 4900
@@
 F 0 "R202" V 4193 4500 50  0000 C CNN
 F 1 "200R" V 4284 4500 50  0000 C CNN
-F 2 "" V 4330 4500 50  0001 C CNN
+F 2 "Resistor_SMD:R_0805_2012Metric" V 4330 4500 50  0001 C CNN
 F 3 "~" H 4400 4500 50  0001 C CNN
 	1    4400 4500
@@
 F 0 "R207" V 4850 4650 50  0000 C CNN
 F 1 "560R" V 4850 4850 50  0000 C CNN
-F 2 "" V 4880 4750 50  0001 C CNN
+F 2 "Resistor_SMD:R_0805_2012Metric" V 4880 4750 50  0001 C CNN
 F 3 "~" H 4950 4750 50  0001 C CNN
 	1    4950 4750
@@
 F 0 "R206" V 4850 4450 50  0000 C CNN
 F 1 "680R" V 4850 4650 50  0000 C CNN
-F 2 "" V 4880 4550 50  0001 C CNN
+F 2 "Resistor_SMD:R_0805_2012Metric" V 4880 4550 50  0001 C CNN
 F 3 "~" H 4950 4550 50  0001 C CNN
 	1    4950 4550
@@
 F 0 "R205" V 4850 4250 50  0000 C CNN
 F 1 "1K" V 4850 4450 50  0000 C CNN
-F 2 "" V 4880 4350 50  0001 C CNN
+F 2 "Resistor_SMD:R_0805_2012Metric" V 4880 4350 50  0001 C CNN
 F 3 "~" H 4950 4350 50  0001 C CNN
 	1    4950 4350
@@
 F 0 "R204" V 4850 4050 50  0000 C CNN
 F 1 "1K5" V 4850 4250 50  0000 C CNN
-F 2 "" V 4880 4150 50  0001 C CNN
+F 2 "Resistor_SMD:R_0805_2012Metric" V 4880 4150 50  0001 C CNN
 F 3 "~" H 4950 4150 50  0001 C CNN
 	1    4950 4150
@@
 F 0 "SW201" H 5750 4817 50  0000 C CNN
 F 1 "Gain_Select" H 5750 4726 50  0000 C CNN
-F 2 "" H 5750 4350 50  0001 C CNN
+F 2 "Package_DIP:SMDIP-8_W7.62mm" H 5750 4350 50  0001 C CNN
 F 3 "~" H 5750 4350 50  0001 C CNN
 	1    5750 4350
@@
 F 0 "R208" V 6843 3250 50  0000 C CNN
 F 1 "47R" V 6934 3250 50  0000 C CNN
-F 2 "" V 6980 3250 50  0001 C CNN
+F 2 "Resistor_SMD:R_0805_2012Metric" V 6980 3250 50  0001 C CNN
 F 3 "~" H 7050 3250 50  0001 C CNN
 	1    7050 3250
@@
 F 0 "L201" V 7369 3250 50  0000 C CNN
 F 1 "680uH" V 7460 3250 50  0000 C CNN
-F 2 "" H 7550 3250 50  0001 C CNN
+F 2 "Inductor_SMD:L_0805_2012Metric" H 7550 3250 50  0001 C CNN
 F 3 "~" H 7550 3250 50  0001 C CNN
 	1    7550 3250
@@
 F 0 "L202" V 7969 3250 50  0000 C CNN
 F 1 "560uH" V 8060 3250 50  0000 C CNN
-F 2 "" H 8150 3250 50  0001 C CNN
+F 2 "Inductor_SMD:L_0805_2012Metric" H 8150 3250 50  0001 C CNN
 F 3 "~" H 8150 3250 50  0001 C CNN
 	1    8150 3250
@@
 F 0 "C206" V 7248 2900 50  0000 C CNN
 F 1 "33pF" V 7339 2900 50  0000 C CNN
-F 2 "" H 7538 2750 50  0001 C CNN
+F 2 "Capacitor_SMD:C_0805_2012Metric" H 7538 2750 50  0001 C CNN
 F 3 "~" H 7500 2900 50  0001 C CNN
 	1    7500 2900
@@
 F 0 "C208" V 7948 2900 50  0000 C CNN
 F 1 "100pF" V 8039 2900 50  0000 C CNN
-F 2 "" H 8238 2750 50  0001 C CNN
+F 2 "Capacitor_SMD:C_0805_2012Metric" H 8238 2750 50  0001 C CNN
 F 3 "~" H 8200 2900 50  0001 C CNN
 	1    8200 2900
@@
 F 0 "C205" V 6998 3650 50  0000 C CNN
 F 1 "330pF" V 7089 3650 50  0000 C CNN
-F 2 "" H 7288 3500 50  0001 C CNN
+F 2 "Capacitor_SMD:C_0805_2012Metric" H 7288 3500 50  0001 C CNN
 F 3 "~" H 7250 3650 50  0001 C CNN
 	1    7250 3650
@@
 F 0 "C207" V 7598 3650 50  0000 C CNN
 F 1 "470pF" V 7689 3650 50  0000 C CNN
-F 2 "" H 7888 3500 50  0001 C CNN
+F 2 "Capacitor_SMD:C_0805_2012Metric" H 7888 3500 50  0001 C CNN
 F 3 "~" H 7850 3650 50  0001 C CNN
 	1    7850 3650
@@
 F 0 "C209" V 8198 3650 50  0000 C CNN
 F 1 "270pF" V 8289 3650 50  0000 C CNN
-F 2 "" H 8488 3500 50  0001 C CNN
+F 2 "Capacitor_SMD:C_0805_2012Metric" H 8488 3500 50  0001 C CNN
 F 3 "~" H 8450 3650 50  0001 C CNN
 	1    8450 3650
@@
 F 0 "R209" V 8493 3250 50  0000 C CNN
 F 1 "47R" V 8584 3250 50  0000 C CNN
-F 2 "" V 8630 3250 50  0001 C CNN
+F 2 "Resistor_SMD:R_0805_2012Metric" V 8630 3250 50  0001 C CNN
 F 3 "~" H 8700 3250 50  0001 C CNN
 	1    8700 3250
@@
 	6150 3250 6900 3250
 Connection ~ 6150 3250
-Text HLabel 9050 3250 2    50   Output ~ 0
+Text HLabel 9250 3250 2    50   Output ~ 0
 RF_OUT
 Wire Wire Line
-	8850 3250 9050 3250
+	8850 3250 9250 3250
 $Comp
 L Device:C C203
@@
 F 0 "C203" V 5298 7050 50  0000 C CNN
 F 1 "100nF" V 5389 7050 50  0000 C CNN
-F 2 "" H 5588 6900 50  0001 C CNN
+F 2 "Capacitor_SMD:C_0805_2012Metric" H 5588 6900 50  0001 C CNN
 F 3 "~" H 5550 7050 50  0001 C CNN
 	1    5550 7050
@@
 F 0 "C204" H 6118 7096 50  0000 L CNN
 F 1 "2.2uF Tant" H 6118 7005 50  0000 L CNN
-F 2 "" H 6038 6900 50  0001 C CNN
+F 2 "Capacitor_Tantalum_SMD:CP_EIA-3216-18_Kemet-A" H 6038 6900 50  0001 C CNN
 F 3 "~" H 6000 7050 50  0001 C CNN
 	1    6000 7050
@@
 	1    0    0    -1
 $EndComp
+Wire Notes Line
+	6750 2350 6750 4400
+Wire Notes Line
+	9000 4400 9000 2350
+Wire Notes Line
+	9000 2350 6750 2350
+Wire Notes Line
+	6750 4400 9000 4400
+Text Notes 6800 2450 0    50   ~ 0
+2N Elliptic Filter (14 MHz low-pass)
+Text Notes 6800 4350 0    50   ~ 0
+Filter capactors should be 5% tolerance
+Text Notes 2050 4950 0    50   ~ 0
+Note:\nThe cable terminating resistor should\ntake into account the parallel resistance of\nthe dividing network:\n\n1000 / 2 = 500 Ohms\n\nRtotal = R1 x R2 / (R1 + R2)\n(500 * 56) / (500 + 56) = 50.36 Ohms
 $EndSCHEMATC

Commit message: Work on the ADS825 module to determine the overall module dimensions and mounting
Parts:
- SW201: footprint Package_DIP:SMDIP-8_W7.62mm -> Button_Switch_SMD:SW_DIP_SPSTx04_Slide_Copal_CHS-04B_W7.62mm_P1.27mm
Changed lines of the file:
@@
 F 0 "SW201" H 5750 4817 50  0000 C CNN
 F 1 "Gain_Select" H 5750 4726 50  0000 C CNN
-F 2 "Package_DIP:SMDIP-8_W7.62mm" H 5750 4350 50  0001 C CNN
+F 2 "Button_Switch_SMD:SW_DIP_SPSTx04_Slide_Copal_CHS-04B_W7.62mm_P1.27mm" H 5750 4350 50  0001 C CNN
 F 3 "~" H 5750 4350 50  0001 C CNN
 	1    5750 4350

Commit message: Added ADC module complete with routing
Parts:
- J201: footprint Connector_Coaxial:SMA_Amphenol_132289_EdgeMount -> digikey-footprints:RF_SMA_RightAngle_5-1814400-1
Changed lines of the file:
@@
 F 0 "J201" H 2828 3388 50  0000 C CNN
 F 1 "RF_In_50R" H 2828 3297 50  0000 C CNN
-F 2 "Connector_Coaxial:SMA_Amphenol_132289_EdgeMount" H 2900 3150 50  0001 C CNN
+F 2 "digikey-footprints:RF_SMA_RightAngle_5-1814400-1" H 2900 3150 50  0001 C CNN
 F 3 " ~" H 2900 3150 50  0001 C CNN
 	1    2900 3150
