File: Hardware/DomesdayDuplicator-module-ADS825/trigger-input.sch (KiCad schematic (older format))
At the start: 8 parts, among them J501 Trigger_In_50R, U501 TLV3501

Commit message: Added DdD base DE0-Nano connections and part mapping for ADS825 module
Parts:
- C501: footprint (none) -> Capacitor_SMD:C_0805_2012Metric
- C502: footprint (none) -> Capacitor_Tantalum_SMD:CP_EIA-3216-18_Kemet-A
- J501: footprint (none) -> Connector_Coaxial:SMA_Amphenol_132289_EdgeMount
- R501, R502, R503: footprint (none) -> Resistor_SMD:R_0805_2012Metric
- RV501: footprint (none) -> Potentiometer_SMD:Potentiometer_Bourns_3314G_Vertical
Other:
- note added: "Note: The potentiometer sets the Vref trigger\npoint between +5V and 0V"
Changed lines of the file:
@@
 F 0 "J501" H 4478 3588 50  0000 C CNN
 F 1 "Trigger_In_50R" H 4478 3497 50  0000 C CNN
-F 2 "" H 4550 3350 50  0001 C CNN
+F 2 "Connector_Coaxial:SMA_Amphenol_132289_EdgeMount" H 4550 3350 50  0001 C CNN
 F 3 " ~" H 4550 3350 50  0001 C CNN
 	1    4550 3350
@@
 F 0 "R501" V 4993 3350 50  0000 C CNN
 F 1 "47R" V 5084 3350 50  0000 C CNN
-F 2 "" V 5130 3350 50  0001 C CNN
+F 2 "Resistor_SMD:R_0805_2012Metric" V 5130 3350 50  0001 C CNN
 F 3 "~" H 5200 3350 50  0001 C CNN
 	1    5200 3350
@@
 F 0 "R503" V 6207 4350 50  0000 C CNN
 F 1 "10K" V 6116 4350 50  0000 C CNN
-F 2 "" V 5930 4350 50  0001 C CNN
+F 2 "Resistor_SMD:R_0805_2012Metric" V 5930 4350 50  0001 C CNN
 F 3 "~" H 6000 4350 50  0001 C CNN
 	1    6000 4350
@@
 F 0 "R502" V 5457 4350 50  0000 C CNN
 F 1 "47R" V 5366 4350 50  0000 C CNN
-F 2 "" V 5180 4350 50  0001 C CNN
+F 2 "Resistor_SMD:R_0805_2012Metric" V 5180 4350 50  0001 C CNN
 F 3 "~" H 5250 4350 50  0001 C CNN
 	1    5250 4350
@@
 F 0 "C501" H 5665 7096 50  0000 L CNN
 F 1 "100nF" H 5665 7005 50  0000 L CNN
-F 2 "" H 5588 6900 50  0001 C CNN
+F 2 "Capacitor_SMD:C_0805_2012Metric" H 5588 6900 50  0001 C CNN
 F 3 "~" H 5550 7050 50  0001 C CNN
 	1    5550 7050
@@
 F 0 "C502" H 6118 7096 50  0000 L CNN
 F 1 "2.2uF Tant" H 6118 7005 50  0000 L CNN
-F 2 "" H 6038 6900 50  0001 C CNN
+F 2 "Capacitor_Tantalum_SMD:CP_EIA-3216-18_Kemet-A" H 6038 6900 50  0001 C CNN
 F 3 "~" H 6000 7050 50  0001 C CNN
 	1    6000 7050
@@
 F 0 "RV501" H 4481 4396 50  0000 R CNN
 F 1 "10K" H 4481 4305 50  0000 R CNN
-F 2 "" H 4550 4350 50  0001 C CNN
+F 2 "Potentiometer_SMD:Potentiometer_Bourns_3314G_Vertical" H 4550 4350 50  0001 C CNN
 F 3 "~" H 4550 4350 50  0001 C CNN
 	1    4550 4350
@@
 	1    0    0    -1
 $EndComp
+Text Notes 4200 5100 0    50   ~ 0
+Note: The potentiometer sets the Vref trigger\npoint between +5V and 0V
 $EndSCHEMATC

Commit message: Added ADC module complete with routing
Parts:
- J501: footprint Connector_Coaxial:SMA_Amphenol_132289_EdgeMount -> digikey-footprints:RF_SMA_RightAngle_5-1814400-1
Changed lines of the file:
@@
 F 0 "J501" H 4478 3588 50  0000 C CNN
 F 1 "Trigger_In_50R" H 4478 3497 50  0000 C CNN
-F 2 "Connector_Coaxial:SMA_Amphenol_132289_EdgeMount" H 4550 3350 50  0001 C CNN
+F 2 "digikey-footprints:RF_SMA_RightAngle_5-1814400-1" H 4550 3350 50  0001 C CNN
 F 3 " ~" H 4550 3350 50  0001 C CNN
 	1    4550 3350
